File: ESP32-S3-MegaMultiFunction/OccupancyDetectors.sch (KiCad schematic (older format))
At the start: 70 parts, among them J901 OC 1-4, J902 OC 5-8, U901 LM339, U902 LM339, U903 LM339, U904 LM339

Commit message: Fix footprint for OC Diodes.
Parts:
- D901, D902, D903, D904, D905, D906, D907, D908, D913, D914, D915, D916, D917, D918, D919, D920: footprint Diodes_SMD:D_SOD-123 -> Diodes_SMD:D_SOD-323
Changed lines of the file:
@@
 F 0 "D901" H 2200 1950 50  0000 C CNN
 F 1 "1N4148" H 2300 1750 50  0000 C CNN
-F 2 "Diodes_SMD:D_SOD-123" H 2300 1850 50  0001 C CNN
+F 2 "Diodes_SMD:D_SOD-323" H 2300 1850 50  0001 C CNN
 F 3 "" H 2300 1850 50  0001 C CNN
 F 4 "750-1N4148WS-HF" H 2300 1850 60  0001 C CNN "Mouser Part Number"
@@
 F 0 "D905" H 2400 1950 50  0000 C CNN
 F 1 "1N4148" H 2500 1750 50  0000 C CNN
-F 2 "Diodes_SMD:D_SOD-123" H 2500 1850 50  0001 C CNN
+F 2 "Diodes_SMD:D_SOD-323" H 2500 1850 50  0001 C CNN
 F 3 "" H 2500 1850 50  0001 C CNN
 F 4 "750-1N4148WS-HF" H 2500 1850 60  0001 C CNN "Mouser Part Number"
@@
 F 0 "D902" H 2200 3250 50  0000 C CNN
 F 1 "1N4148" H 2300 3050 50  0000 C CNN
-F 2 "Diodes_SMD:D_SOD-123" H 2300 3150 50  0001 C CNN
+F 2 "Diodes_SMD:D_SOD-323" H 2300 3150 50  0001 C CNN
 F 3 "" H 2300 3150 50  0001 C CNN
 F 4 "750-1N4148WS-HF" H 2300 3150 60  0001 C CNN "Mouser Part Number"
@@
 F 0 "D906" H 2400 3250 50  0000 C CNN
 F 1 "1N4148" H 2500 3050 50  0000 C CNN
-F 2 "Diodes_SMD:D_SOD-123" H 2500 3150 50  0001 C CNN
+F 2 "Diodes_SMD:D_SOD-323" H 2500 3150 50  0001 C CNN
 F 3 "" H 2500 3150 50  0001 C CNN
 F 4 "750-1N4148WS-HF" H 2500 3150 60  0001 C CNN "Mouser Part Number"
@@
 F 0 "D903" H 2200 4450 50  0000 C CNN
 F 1 "1N4148" H 2300 4250 50  0000 C CNN
-F 2 "Diodes_SMD:D_SOD-123" H 2300 4350 50  0001 C CNN
+F 2 "Diodes_SMD:D_SOD-323" H 2300 4350 50  0001 C CNN
 F 3 "" H 2300 4350 50  0001 C CNN
 F 4 "750-1N4148WS-HF" H 2300 4350 60  0001 C CNN "Mouser Part Number"
@@
 F 0 "D907" H 2400 4450 50  0000 C CNN
 F 1 "1N4148" H 2500 4250 50  0000 C CNN
-F 2 "Diodes_SMD:D_SOD-123" H 2500 4350 50  0001 C CNN
+F 2 "Diodes_SMD:D_SOD-323" H 2500 4350 50  0001 C CNN
 F 3 "" H 2500 4350 50  0001 C CNN
 F 4 "750-1N4148WS-HF" H 2500 4350 60  0001 C CNN "Mouser Part Number"
@@
 F 0 "D904" H 2200 5850 50  0000 C CNN
 F 1 "1N4148" H 2300 5650 50  0000 C CNN
-F 2 "Diodes_SMD:D_SOD-123" H 2300 5750 50  0001 C CNN
+F 2 "Diodes_SMD:D_SOD-323" H 2300 5750 50  0001 C CNN
 F 3 "" H 2300 5750 50  0001 C CNN
 F 4 "750-1N4148WS-HF" H 2300 5750 60  0001 C CNN "Mouser Part Number"
@@
 F 0 "D908" H 2400 5850 50  0000 C CNN
 F 1 "1N4148" H 2500 5650 50  0000 C CNN
-F 2 "Diodes_SMD:D_SOD-123" H 2500 5750 50  0001 C CNN
+F 2 "Diodes_SMD:D_SOD-323" H 2500 5750 50  0001 C CNN
 F 3 "" H 2500 5750 50  0001 C CNN
 F 4 "750-1N4148WS-HF" H 2500 5750 60  0001 C CNN "Mouser Part Number"
@@
 F 0 "D913" H 7275 1750 50  0000 C CNN
 F 1 "1N4148" H 7375 1550 50  0000 C CNN
-F 2 "Diodes_SMD:D_SOD-123" H 7375 1650 50  0001 C CNN
+F 2 "Diodes_SMD:D_SOD-323" H 7375 1650 50  0001 C CNN
 F 3 "" H 7375 1650 50  0001 C CNN
 F 4 "750-1N4148WS-HF" H 7375 1650 60  0001 C CNN "Mouser Part Number"
@@
 F 0 "D917" H 7475 1750 50  0000 C CNN
 F 1 "1N4148" H 7575 1550 50  0000 C CNN
-F 2 "Diodes_SMD:D_SOD-123" H 7575 1650 50  0001 C CNN
+F 2 "Diodes_SMD:D_SOD-323" H 7575 1650 50  0001 C CNN
 F 3 "" H 7575 1650 50  0001 C CNN
 F 4 "750-1N4148WS-HF" H 7575 1650 60  0001 C CNN "Mouser Part Number"
@@
 F 0 "D914" H 7275 3050 50  0000 C CNN
 F 1 "1N4148" H 7375 2850 50  0000 C CNN
-F 2 "Diodes_SMD:D_SOD-123" H 7375 2950 50  0001 C CNN
+F 2 "Diodes_SMD:D_SOD-323" H 7375 2950 50  0001 C CNN
 F 3 "" H 7375 2950 50  0001 C CNN
 F 4 "750-1N4148WS-HF" H 7375 2950 60  0001 C CNN "Mouser Part Number"
@@
 F 0 "D918" H 7475 3050 50  0000 C CNN
 F 1 "1N4148" H 7575 2850 50  0000 C CNN
-F 2 "Diodes_SMD:D_SOD-123" H 7575 2950 50  0001 C CNN
+F 2 "Diodes_SMD:D_SOD-323" H 7575 2950 50  0001 C CNN
 F 3 "" H 7575 2950 50  0001 C CNN
 F 4 "750-1N4148WS-HF" H 7575 2950 60  0001 C CNN "Mouser Part Number"
@@
 F 0 "D915" H 7275 4250 50  0000 C CNN
 F 1 "1N4148" H 7375 4050 50  0000 C CNN
-F 2 "Diodes_SMD:D_SOD-123" H 7375 4150 50  0001 C CNN
+F 2 "Diodes_SMD:D_SOD-323" H 7375 4150 50  0001 C CNN
 F 3 "" H 7375 4150 50  0001 C CNN
 F 4 "750-1N4148WS-HF" H 7375 4150 60  0001 C CNN "Mouser Part Number"
@@
 F 0 "D919" H 7475 4250 50  0000 C CNN
 F 1 "1N4148" H 7575 4050 50  0000 C CNN
-F 2 "Diodes_SMD:D_SOD-123" H 7575 4150 50  0001 C CNN
+F 2 "Diodes_SMD:D_SOD-323" H 7575 4150 50  0001 C CNN
 F 3 "" H 7575 4150 50  0001 C CNN
 F 4 "750-1N4148WS-HF" H 7575 4150 60  0001 C CNN "Mouser Part Number"
@@
 F 0 "D916" H 7275 5650 50  0000 C CNN
 F 1 "1N4148" H 7375 5450 50  0000 C CNN
-F 2 "Diodes_SMD:D_SOD-123" H 7375 5550 50  0001 C CNN
+F 2 "Diodes_SMD:D_SOD-323" H 7375 5550 50  0001 C CNN
 F 3 "" H 7375 5550 50  0001 C CNN
 F 4 "750-1N4148WS-HF" H 7375 5550 60  0001 C CNN "Mouser Part Number"
@@
 F 0 "D920" H 7475 5650 50  0000 C CNN
 F 1 "1N4148" H 7575 5450 50  0000 C CNN
-F 2 "Diodes_SMD:D_SOD-123" H 7575 5550 50  0001 C CNN
+F 2 "Diodes_SMD:D_SOD-323" H 7575 5550 50  0001 C CNN
 F 3 "" H 7575 5550 50  0001 C CNN
 F 4 "750-1N4148WS-HF" H 7575 5550 60  0001 C CNN "Mouser Part Number"
