File: ESP32-16LedDriver/CAN_Transeiver.sch (KiCad schematic (older format))
At the start: 14 parts, among them J1 RJ45, J2 RJ45, T1 + 15 in -, T2 + 15 out -, U1 TCAN332DR, U2 SN65HVD233-HT

Commit message: Cleanup and refactor.
Parts:
- C1, C3: symbol C -> C-RESCUE-ESP32-16LedDriver
- C2: symbol CP1 -> CP1-RESCUE-ESP32-16LedDriver
- R1, R2: symbol R -> R-RESCUE-ESP32-16LedDriver
Changed lines of the file:
@@
 EESchema Schematic File Version 2
+LIBS:ESP32-16LedDriver-rescue
 LIBS:power
 LIBS:device
@@
 LIBS:memory
 LIBS:xilinx
-LIBS:special
 LIBS:microcontrollers
 LIBS:dsp
@@
 LIBS:tbd62x83a
 LIBS:ESP32-16LedDriver-cache
-EELAYER 27 0
+EELAYER 25 0
 EELAYER END
 $Descr A4 11693 8268
@@
 $EndComp
 $Comp
-L GND #PWR07
+L GND-RESCUE-ESP32-16LedDriver #PWR07
 U 1 1 5C828CBC
 P 4100 3800
@@
 $EndComp
 $Comp
-L GND #PWR08
+L GND-RESCUE-ESP32-16LedDriver #PWR08
 U 1 1 5C828CCB
 P 4100 4950
@@
 Connection ~ 3750 4400
 $Comp
-L C C1
+L C-RESCUE-ESP32-16LedDriver C1
 U 1 1 5C828DA1
 P 4650 3800
+AR Path="/5C828DA1" Ref="C1"  Part="1"
+AR Path="/5C828AE5/5C828DA1" Ref="C1"  Part="1"
 F 0 "C1" H 4650 3900 40  0000 L CNN
 F 1 ".1 uf" H 4656 3715 40  0000 L CNN
@@
 $EndComp
 $Comp
-L CP1 C2
+L CP1-RESCUE-ESP32-16LedDriver C2
 U 1 1 5C828DB0
 P 5000 3800
@@
 CANL
 $Comp
-L R R1
+L R-RESCUE-ESP32-16LedDriver R1
 U 1 1 5C828F93
 P 5850 3650
@@
 $EndComp
 $Comp
-L R R2
+L R-RESCUE-ESP32-16LedDriver R2
 U 1 1 5C828FA2
 P 6550 3650
@@
 	6700 4150 6600 4150
 $Comp
-L C C3
+L C-RESCUE-ESP32-16LedDriver C3
 U 1 1 5C8290C3
 P 6200 4750
+AR Path="/5C8290C3" Ref="C3"  Part="1"
+AR Path="/5C828AE5/5C8290C3" Ref="C3"  Part="1"
 F 0 "C3" H 6200 4850 40  0000 L CNN
 F 1 "47 nf" H 6206 4665 40  0000 L CNN
@@
 $EndComp
 $Comp
-L GND #PWR09
+L GND-RESCUE-ESP32-16LedDriver #PWR09
 U 1 1 5C8290D2
 P 6200 5100
@@
 	7450 3000 7450 5050
 $Comp
-L GND #PWR010
+L GND-RESCUE-ESP32-16LedDriver #PWR010
 U 1 1 5C8295F7
 P 6750 2650
