File: ESP32-S3-MultiFunction/OccDetect4.sch (KiCad schematic (older format))
At the start: 35 parts, among them U601 LM339, U602 LM339

Commit message: Fix footprint for OC Diodes.
Parts:
- D601, D602, D603, D604, D605, D606, D607, D608: footprint Diodes_SMD:D_SOD-123 -> Diodes_SMD:D_SOD-323
Changed lines of the file:
@@
 F 0 "D601" H 2200 1950 50  0000 C CNN
 F 1 "1N4148" H 2300 1750 50  0000 C CNN
-F 2 "Diodes_SMD:D_SOD-123" H 2300 1850 50  0001 C CNN
+F 2 "Diodes_SMD:D_SOD-323" H 2300 1850 50  0001 C CNN
 F 3 "" H 2300 1850 50  0001 C CNN
 F 4 "750-1N4148WS-HF" H 2300 1850 60  0001 C CNN "Mouser Part Number"
@@
 F 0 "D605" H 2400 1950 50  0000 C CNN
 F 1 "1N4148" H 2500 1750 50  0000 C CNN
-F 2 "Diodes_SMD:D_SOD-123" H 2500 1850 50  0001 C CNN
+F 2 "Diodes_SMD:D_SOD-323" H 2500 1850 50  0001 C CNN
 F 3 "" H 2500 1850 50  0001 C CNN
 F 4 "750-1N4148WS-HF" H 2500 1850 60  0001 C CNN "Mouser Part Number"
@@
 F 0 "D602" H 2200 3250 50  0000 C CNN
 F 1 "1N4148" H 2300 3050 50  0000 C CNN
-F 2 "Diodes_SMD:D_SOD-123" H 2300 3150 50  0001 C CNN
+F 2 "Diodes_SMD:D_SOD-323" H 2300 3150 50  0001 C CNN
 F 3 "" H 2300 3150 50  0001 C CNN
 F 4 "750-1N4148WS-HF" H 2300 3150 60  0001 C CNN "Mouser Part Number"
@@
 F 0 "D606" H 2400 3250 50  0000 C CNN
 F 1 "1N4148" H 2500 3050 50  0000 C CNN
-F 2 "Diodes_SMD:D_SOD-123" H 2500 3150 50  0001 C CNN
+F 2 "Diodes_SMD:D_SOD-323" H 2500 3150 50  0001 C CNN
 F 3 "" H 2500 3150 50  0001 C CNN
 F 4 "750-1N4148WS-HF" H 2500 3150 60  0001 C CNN "Mouser Part Number"
@@
 F 0 "D603" H 2200 4450 50  0000 C CNN
 F 1 "1N4148" H 2300 4250 50  0000 C CNN
-F 2 "Diodes_SMD:D_SOD-123" H 2300 4350 50  0001 C CNN
+F 2 "Diodes_SMD:D_SOD-323" H 2300 4350 50  0001 C CNN
 F 3 "" H 2300 4350 50  0001 C CNN
 F 4 "750-1N4148WS-HF" H 2300 4350 60  0001 C CNN "Mouser Part Number"
@@
 F 0 "D607" H 2400 4450 50  0000 C CNN
 F 1 "1N4148" H 2500 4250 50  0000 C CNN
-F 2 "Diodes_SMD:D_SOD-123" H 2500 4350 50  0001 C CNN
+F 2 "Diodes_SMD:D_SOD-323" H 2500 4350 50  0001 C CNN
 F 3 "" H 2500 4350 50  0001 C CNN
 F 4 "750-1N4148WS-HF" H 2500 4350 60  0001 C CNN "Mouser Part Number"
@@
 F 0 "D604" H 2200 5850 50  0000 C CNN
 F 1 "1N4148" H 2300 5650 50  0000 C CNN
-F 2 "Diodes_SMD:D_SOD-123" H 2300 5750 50  0001 C CNN
+F 2 "Diodes_SMD:D_SOD-323" H 2300 5750 50  0001 C CNN
 F 3 "" H 2300 5750 50  0001 C CNN
 F 4 "750-1N4148WS-HF" H 2300 5750 60  0001 C CNN "Mouser Part Number"
@@
 F 0 "D608" H 2400 5850 50  0000 C CNN
 F 1 "1N4148" H 2500 5650 50  0000 C CNN
-F 2 "Diodes_SMD:D_SOD-123" H 2500 5750 50  0001 C CNN
+F 2 "Diodes_SMD:D_SOD-323" H 2500 5750 50  0001 C CNN
 F 3 "" H 2500 5750 50  0001 C CNN
 F 4 "750-1N4148WS-HF" H 2500 5750 60  0001 C CNN "Mouser Part Number"
