File: ESP32-OctalServo/ESP32-OctalServo.kicad_pcb (KiCad board)
At the start: 2 copper layers, 66 x 91.4 mm, 33 parts, among them J101 Servo Power, J102 Servo 1, J103 Servo 2, J104 Servo 3, J105 Servo 4, J106 Servo 5, J107 Servo 6, J108 Servo 7, J109 Servo 8, J301 RJ45, J302 RJ45, T301 - 15 in +, T302 - 15 out +, U201 ESP32_DEVKIT_C, U202 TTGO-T1, U301 TCAN332DR, U401 LM2574N-5.0

Commit message: Finalize the design.
Parts:
- added ?: , DWSLogoBCU:DWSLogoBCU, F.Cu at (184.8, 67.3)
- added G***: LCC, LCC_LOGO:LCC_LOGO_4.5x4.5, F.Cu at (169.5, 128.9)
- added REF**: PowerLabel-100, PowerLabels:PowerLabel-100, F.Cu at (176.5, 139.1)
- added REF***: ESD-Logo_8.9x8mm_SilkScreen, Symbols:ESD-Logo_8.9x8mm_SilkScreen, F.Cu at (161.3, 66.7)
- added REF***: KiCad-Logo2_8mm_SilkScreen, Symbols:KiCad-Logo2_8mm_SilkScreen, F.Cu at (176.5, 67.3)
- added REF***: OSHW-Logo_5.7x6mm_SilkScreen, Symbols:OSHW-Logo_5.7x6mm_SilkScreen, F.Cu at (190.5, 67.3)
- added REF***: WEEE-Logo_4.2x6mm_SilkScreen, Symbols:WEEE-Logo_4.2x6mm_SilkScreen, F.Cu at (181.0, 129.5)
- J101: value Servo Power -> + 5V Servo -
Other:
- board text added: "(C) 2022 Robert Heller D/B/A Deepwoods Software ESP32-OctalServo"

Commit message: Update PS.
Parts:
- removed D401: CMSH1-60 TR13, Diodes_SMD:D_SMB
- added C403: 22uf, Capacitors_SMD:C_0603, F.Cu at (149.3, 114.3)
- added C404: 22uf, Capacitors_SMD:C_0603, F.Cu at (149.3, 111.8)
- C401: value 220 uf 25V -> 10uf; footprint Capacitors_SMD:CP_Elec_8x10 -> Capacitors_SMD:CP_Elec_5x5.3
- C402: value 22 uf 100V -> 100nf; footprint Capacitors_SMD:CP_Elec_8x10 -> Capacitors_SMD:C_0603
- L401: value 330 uh -> 4.7uH; footprint SRN1060:SRN1060 -> Inductors_SMD:L_7.3x7.3_H4.5
- U401: value LM2574N-5.0 -> AP63205; footprint SOIC_Wide:SOIC-14_7.4x8.7mm_Pitch1.27mm -> TO_SOT_Packages_SMD:TSOT-23-6_MK06A
- moved C401 40.6 mm to (155.2, 119.4), turned to 0 degrees
- moved L401 11.0 mm to (153.7, 103.5), turned to 270 degrees
- moved U401 8.65 mm to (153.3, 113.0)
- moved C402 8.26 mm to (152.5, 109.2)
Connections:
- C401 pad 1: +5V -> CAN +12V
- C402 pad 1: CAN +12V -> Net-(C402-Pad1)
- C402 pad 2: GND -> Net-(C402-Pad2)
- L401 pad 1: Net-(D401-Pad1) -> +5V
- L401 pad 2: +5V -> Net-(C402-Pad2)
- U401 pad 1: Net-(U401-Pad1) -> +5V
- U401 pad 2: Net-(U401-Pad2) -> CAN +12V
- U401 pad 3: +5V -> CAN +12V
- U401 pad 5: GND -> Net-(C402-Pad2)
- U401 pad 6: GND -> Net-(C402-Pad1)
Routing:
- net +5V: track 107.5 -> 53.6 mm, vias 4 -> 2
- net GND: track 70.6 -> 32.9 mm, vias 5 -> 6
- net CAN +12V: track 118.7 -> 90.7 mm, vias 7 -> 5
- net Net-(D401-Pad1): track 21.2 -> 0.00 mm
- net Net-(C402-Pad2): track 0.00 -> 5.15 mm
- net Net-(C402-Pad1): track 0.00 -> 2.72 mm
- added copper zone on F.Cu, net +5V
