File: ESP32-OctalServo/ESP32-OctalServo.sch (KiCad schematic (older format))
At the start: 9 parts, among them J101 Servo Power, J102 Servo 1, J103 Servo 2, J104 Servo 3, J105 Servo 4, J106 Servo 5, J107 Servo 6, J108 Servo 7, J109 Servo 8

Commit message: Finalize the design.
Parts:
- J101: value Servo Power -> + 5V Servo -
Changed lines of the file:
@@
 P 7125 6275
 F 0 "J101" H 7125 6375 50  0000 C CNN
-F 1 "Servo Power" H 7125 6075 50  0000 C CNN
+F 1 "+ 5V Servo -" H 7125 6075 50  0000 C CNN
 F 2 "Connectors_Terminal_Blocks:TerminalBlock_Pheonix_PT-3.5mm_2pol" H 7125 6275 50  0001 C CNN
 F 3 "" H 7125 6275 50  0001 C CNN
