File: ESP32-T7S3-MultiFunction/ESP32-T7S3-MultiFunction.kicad_pcb (KiCad board)
At the start: 2 copper layers, 99.1 x 125.7 mm, 130 parts, among them J501 -SM+, J801 RJ45, J802 RJ45, P701 A7 A6 A5 A4 A3 A2 A1 A0 C, P702 B7 B6 B5 B4 B3 B2 B1 B0 C, T701 + 12V -, T801 - 15 in +, T802 - 15 out +, U201 TTGO-T7_S3-V1.1, U301 LM2574N-3.3, U401 TC4426, U402 TC4426, U403 74HCT14, U501 74HCT00, U502 74HCT00, U503 TC4428, U504 TC4428, U505 TC4428, U506 TC4428, U601 LM339, U602 LM339, U701 PCA9685, U702 TBD62X83A, U703 TBD62X83A, U801 TCAN332DR

Commit message: Finalize T7S3 MultiFunction.
Parts:
- removed D1, D3: DFLS240-7, Diodes_SMD:D_PowerDI-123
- removed D301: CMSH1-60 TR13, Diodes_SMD:D_SMB
- added C303: 22uf, Capacitors_SMD:C_0603, F.Cu at (160.3, 119.1)
- added C304: 22uf, Capacitors_SMD:C_0603, F.Cu at (160.3, 117.5)
- C301: value 220 uf 25V -> 10uf; footprint Capacitors_SMD:CP_Elec_8x10 -> Capacitors_SMD:CP_Elec_5x5.3
- C302: value 22 uf 100V -> 100nf; footprint Capacitors_SMD:CP_Elec_8x10 -> Capacitors_SMD:C_0603
- FD101, FD102: footprint Fiducials:Fiducial_1mm_Dia_2.54mm_Outer_CopperTop -> Fiducials:Fiducial_classic_Small_SilkscreenTop_Type1
- FD103: footprint Fiducials:Fiducial_1mm_Dia_2.54mm_Outer_CopperTop -> Fiducials:Fiducial_classic_Small_SilkscreenTop_Type1; moved to F.Cu
- L301: value 330 uh -> 4.7uH; footprint SRN1060:SRN1060 -> Inductors_SMD:L_7.3x7.3_H4.5
- REF**: footprint PowerLabels:PowerLabel-30Plus -> PowerLabels:PowerLabel-100
- U301: value LM2574N-3.3 -> AP63205; footprint SOIC_Wide:SOIC-14_7.4x8.7mm_Pitch1.27mm -> TO_SOT_Packages_SMD:TSOT-23-6_MK06A
- moved R206 133.2 mm to (141.5, 29.2)
- moved R203 107.0 mm to (140.0, 55.5)
- moved D4 101.7 mm to (116.3, 59.7)
- moved R3 101.6 mm to (118.4, 59.7), turned to 180 degrees
- moved D2 100.5 mm to (116.3, 61.0)
- moved R2 100.3 mm to (118.4, 61.0), turned to 180 degrees
- moved FD101 98.9 mm to (156.2, 37.2)
- moved FD103 86.1 mm to (149.9, 113.3)
- moved FD102 61.4 mm to (121.8, 46.6)
- moved REF*** 26.4 mm to (133.3, 85.1)
- moved C302 25.4 mm to (167.8, 118.5), turned to 270 degrees
- moved C301 12.5 mm to (164.4, 124.7)
- moved U301 11.9 mm to (164.3, 119.1), turned to 0 degrees
- moved L301 11.1 mm to (164.7, 111.4), turned to 0 degrees
Connections:
- C301 pad 1: +3V3 -> CAN +12V
- C302 pad 2: GND -> Net-(C302-Pad2)
- L301 pad 1: Net-(D301-Pad1) -> +5V
- L301 pad 2: +3V3 -> Net-(C302-Pad2)
- U201 pad 1: Net-(U201-Pad1) -> GND
- U201 pad 16: Net-(U201-Pad16) -> +3V3
- U201 pad 22: Net-(U201-Pad22) -> GND
- U201 pad 33: Net-(U201-Pad33) -> GND
- U201 pad 35: Net-(U201-Pad35) -> +5V
- U301 pad 1: Net-(U301-Pad1) -> +5V
- U301 pad 2: Net-(U301-Pad2) -> CAN +12V
- U301 pad 3: +3V3 -> CAN +12V
- U301 pad 5: GND -> Net-(C302-Pad2)
- U301 pad 6: GND -> Net-(C302-Pad1)
Routing:
- net Net-(C302-Pad1): track 153.1 -> 2.31 mm, vias 6 -> 0
- net /Buttons and LEDs/Button4: track 21.8 -> 150.1 mm, vias 2 -> 5
- net /Buttons and LEDs/Button3: track 19.1 -> 140.8 mm, vias 2 -> 5
- net +5V: track 0.00 -> 104.6 mm, vias 0 -> 2
- net /Buttons and LEDs/Button2: track 16.9 -> 112.4 mm, vias 2 -> 5
- net /CAN Tranceiver/CAN_RX: track 13.0 -> 105.1 mm, vias 2 -> 1
- net /ESP32 MCU/GPIO7(OD4): track 10.0 -> 96.1 mm, vias 3 -> 4
- net /CAN Tranceiver/CAN_TX: track 9.08 -> 90.0 mm, vias 2 -> 1
- net /ESP32 MCU/GPIO14(Points3): track 1.36 -> 78.3 mm
- net /ESP32 MCU/GPIO17(LEDS1): track 76.3 -> 148.4 mm, vias 2 -> 6
- net /ESP32 MCU/GPIO44/TXD(OD1): track 42.7 -> 111.9 mm, vias 6 -> 5
- net /ESP32 MCU/GPIO48(OD2): track 41.6 -> 109.1 mm
- net /ESP32 MCU/GPIO43/RXD(Motor4): track 47.6 -> 110.0 mm, vias 1 -> 3
- net /ESP32 MCU/GPIO15(Act1): track 0.00 -> 54.6 mm, vias 0 -> 3
- net /ESP32 MCU/GPIO45(OD3): track 51.5 -> 105.0 mm
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Other:
- board text added: "(c) Copyright 2023 Robert Heller D/B/A Deepwoods Software ESP32-T7S3-MultiFunction board rev D"
- board text removed: "(c) Copyright 2022 Robert Heller D/B/A Deepwoods Software ESP32-S3-MultiFunction board rev C"
