File: ESP32-T7S3-MultiFunction/PowerSupply.sch (KiCad schematic (older format))
At the start: 6 parts, among them U301 LM2574N-3.3

Commit message: Finalize T7S3 MultiFunction.
Parts:
- removed C301: 220 uf 25V, Capacitors_SMD:CP_Elec_8x10, symbol CP1
- removed C302: 22 uf 100V, Capacitors_SMD:CP_Elec_8x10, symbol CP1
- removed D3: DFLS240-7, Diodes_SMD:D_PowerDI-123, symbol D_Schottky
- removed D301: CMSH1-60 TR13, Diodes_SMD:D_SMB, symbol D_Schottky
- removed U301: LM2574N-3.3, SOIC_Wide:SOIC-14_7.4x8.7mm_Pitch1.27mm, symbol LM2574HVM-5.0
- added C301: 10uf, Capacitors_SMD:CP_Elec_5x5.3, symbol CP1_Small
- added C302: 100nf, Capacitors_SMD:C_0603, symbol C_Small
- added C303, C304: 22uf, Capacitors_SMD:C_0603, symbol C_Small
- added U301: AP63205, TO_SOT_Packages_SMD:TSOT-23-6_MK06A, symbol AP63205
- L301: value 330 uh -> 4.7uH; footprint SRN1060:SRN1060 -> Inductors_SMD:L_7.3x7.3_H4.5; Mouser Part Number 652-SRN1060-331M -> 81-B1047AS-4R7NP3
Connections:
- net CAN +12V: now also C301.1, U301.2 (EN), U301.3 (Vin)
- net GND: now also C301.2, C303.2, C304.2, U301.4 (GND)
- net +5V: now reaches L301.1
- net +5V: now also C303.1, C304.1, U301.1 (FB)
- net +3V3: no longer names the net of L301.2
- net +3V3: now also C302.2, U301.5 (SW)
- new net: C302.1, U301.6 (BST)
- no-connect marks 8 -> 0
Changed lines of the file:
@@
 LIBS:gct_usb4105
 LIBS:ESP32_mini
+LIBS:ap63205
 EELAYER 25 0
 EELAYER END
@@
 Comment4 ""
 $EndDescr
+Text GLabel 3350 4600 0    50   Input ~ 0
+CAN +12V
 $Comp
-L LM2574HVM-5.0 U301
-U 1 1 62AF11D9
-P 5200 2800
-F 0 "U301" H 5200 2850 60  0000 C CNN
-F 1 "LM2574N-3.3" H 5200 2950 21  0000 C CNN
-F 2 "SOIC_Wide:SOIC-14_7.4x8.7mm_Pitch1.27mm" H 5200 2800 60  0001 C CNN
-F 3 "~" H 5200 2800 60  0000 C CNN
-F 4 "926-LM2574MX33NOPB" H 5200 2800 60  0001 C CNN "Mouser Part Number"
-	1    5200 2800
+L +5V #PWR07
+U 1 1 63E7CCDF
+P 5600 4700
+F 0 "#PWR07" H 5600 4550 50  0001 C CNN
+F 1 "+5V" H 5600 4840 50  0000 C CNN
+F 2 "" H 5600 4700 50  0001 C CNN
+F 3 "" H 5600 4700 50  0001 C CNN
+	1    5600 4700
 	1    0    0    -1
 $EndComp
 $Comp
-L CP1 C302
-U 1 1 62AF11DA
-P 5950 2900
-F 0 "C302" H 6000 3000 50  0000 L CNN
-F 1 "22 uf 100V" H 6000 2800 50  0000 L CNN
-F 2 "Capacitors_SMD:CP_Elec_8x10" H 5950 2900 60  0001 C CNN
-F 3 "~" H 5950 2900 60  0000 C CNN
-F 4 "647-UUX2A220MNL6GS" H 5950 2900 60  0001 C CNN "Mouser Part Number"
-	1    5950 2900
+L AP63205 U301
+U 1 1 63E7CCE0
+P 4275 4775
+F 0 "U301" H 4275 4775 60  0000 C CNN
+F 1 "AP63205" H 4275 4875 60  0000 C CNN
+F 2 "TO_SOT_Packages_SMD:TSOT-23-6_MK06A" H 4275 4775 60  0001 C CNN
+F 3 "" H 4275 4775 60  0001 C CNN
+F 4 "621-AP63205WU-7" H 4275 4775 60  0001 C CNN "Mouser Part Number"
+	1    4275 4775
 	1    0    0    -1
 $EndComp
 $Comp
-L CP1 C301
-U 1 1 62AF11DB
-P 3700 2800
-F 0 "C301" H 3750 2900 50  0000 L CNN
-F 1 "220 uf 25V" H 3750 2700 50  0000 L CNN
-F 2 "Capacitors_SMD:CP_Elec_8x10" H 3700 2800 60  0001 C CNN
-F 3 "~" H 3700 2800 60  0000 C CNN
-F 4 "647-UWT1E221MNL1GS" H 3700 2800 60  0001 C CNN "Mouser Part Number"
-	1    3700 2800
+L CP1_Small C301
+U 1 1 63E7CCE1
+P 3600 4800
+F 0 "C301" H 3610 4870 50  0000 L CNN
+F 1 "10uf" H 3610 4720 50  0000 L CNN
+F 2 "Capacitors_SMD:CP_Elec_5x5.3" H 3600 4800 50  0001 C CNN
+F 3 "" H 3600 4800 50  0001 C CNN
+F 4 "710-865230542002" H 3600 4800 60  0001 C CNN "Mouser Part Number"
+	1    3600 4800
+	1    0    0    -1
+$EndComp
+$Comp
+L GND #PWR08
+U 1 1 63E7CCE2
+P 3600 5075
+F 0 "#PWR08" H 3600 4825 50  0001 C CNN
+F 1 "GND" H 3600 4925 50  0000 C CNN
+F 2 "" H 3600 5075 50  0001 C CNN
+F 3 "" H 3600 5075 50  0001 C CNN
+	1    3600 5075
+	1    0    0    -1
+$EndComp
+$Comp
+L C_Small C302
+U 1 1 63E7CCE3
+P 4900 4675
+F 0 "C302" H 4910 4745 50  0000 L CNN
+F 1 "100nf" H 4910 4595 50  0000 L CNN
+F 2 "Capacitors_SMD:C_0603" H 4900 4675 50  0001 C CNN
+F 3 "" H 4900 4675 50  0001 C CNN
+F 4 "710-885012206020" H 4900 4675 60  0001 C CNN "Mouser Part Number"
+	1    4900 4675
 	1    0    0    -1
 $EndComp
 $Comp
 L L_Small L301
-U 1 1 62AF11DC
-P 4550 2900
-F 0 "L301" H 4550 3000 50  0000 C CNN
-F 1 "330 uh" H 4550 2850 50  0000 C CNN
-F 2 "SRN1060:SRN1060" H 4550 2900 60  0001 C CNN
-F 3 "~" H 4550 2900 60  0000 C CNN
-F 4 "652-SRN1060-331M" H 4550 2900 60  0001 C CNN "Mouser Part Number"
-	1    4550 2900
+U 1 1 63E7CCE4
+P 5175 4775
+F 0 "L301" H 5205 4815 50  0000 L CNN
+F 1 "4.7uH" H 5205 4735 50  0000 L CNN
+F 2 "Inductors_SMD:L_7.3x7.3_H4.5" H 5175 4775 50  0001 C CNN
+F 3 "" H 5175 4775 50  0001 C CNN
+F 4 "81-B1047AS-4R7NP3" H 5175 4775 60  0001 C CNN "Mouser Part Number"
+	1    5175 4775
 	0    1    1    0
 $EndComp
 $Comp
-L D_Schottky D301
-U 1 1 62AF11DD
-P 4850 3100
-F 0 "D301" H 4850 3200 40  0000 C CNN
-F 1 "CMSH1-60 TR13" H 4850 3000 40  0000 C CNN
-F 2 "Diodes_SMD:D_SMB" H 4850 3100 60  0001 C CNN
-F 3 "~" H 4850 3100 60  0000 C CNN
-F 4 "610-CMSH1-60TR13" H 4850 3100 60  0001 C CNN "Mouser Part Number"
-	1    4850 3100
-	0    1    1    0
-$EndComp
-Wire Wire Line
-	5950 2700 5500 2700
-Wire Wire Line
-	4900 2600 3700 2600
-Wire Wire Line
-	4300 2900 4300 2600
-Connection ~ 4300 2600
-Wire Wire Line
-	4650 2900 4900 2900
-Connection ~ 4850 2900
-Wire Wire Line
-	5950 3050 5950 3150
-Wire Wire Line
-	5950 3150 5150 3150
-Connection ~ 5350 3150
-Connection ~ 5250 3150
-Wire Wire Line
-	5150 3150 5150 3300
-Wire Wire Line
-	5150 3300 3700 3300
-Wire Wire Line
-	3700 3300 3700 2950
-Connection ~ 4850 3300
-$Comp
-L GND #PWR04
-U 1 1 62AF11DE
-P 4850 3400
-F 0 "#PWR04" H 4850 3400 30  0001 C CNN
-F 1 "GND" H 4850 3330 30  0001 C CNN
-F 2 "" H 4850 3400 60  0000 C CNN
-F 3 "" H 4850 3400 60  0000 C CNN
-	1    4850 3400
+L C_Small C303
+U 1 1 63E7CCE5
+P 5375 4875
+F 0 "C303" H 5385 4945 50  0000 L CNN
+F 1 "22uf" H 5385 4795 50  0000 L CNN
+F 2 "Capacitors_SMD:C_0603" H 5375 4875 50  0001 C CNN
+F 3 "" H 5375 4875 50  0001 C CNN
+F 4 "603-CC0603MRX6S5B226" H 5375 4875 60  0001 C CNN "Mouser Part Number"
+	1    5375 4875
 	1    0    0    -1
 $EndComp
 Wire Wire Line
-	3700 2450 3700 2650
+	3350 4600 3850 4600
 Wire Wire Line
-	4850 3250 4850 3400
-Text GLabel 6250 2500 2    50   Input ~ 0
-CAN +12V
-Connection ~ 3700 2600
+	3850 4600 3850 4775
 Wire Wire Line
-	4450 2900 4300 2900
+	3600 4700 3600 4600
+Connection ~ 3600 4600
 Wire Wire Line
-	4850 2950 4850 2900
-Connection ~ 5950 2700
-NoConn ~ 5500 2900
-NoConn ~ 5500 2800
-NoConn ~ 5350 2450
-NoConn ~ 5300 2450
-NoConn ~ 5250 2450
-NoConn ~ 5200 2450
-NoConn ~ 5150 2450
-NoConn ~ 5100 2450
+	3600 4900 3600 5075
+Wire Wire Line
+	4775 4600 4775 4550
+Wire Wire Line
+	4775 4550 4900 4550
+Wire Wire Line
+	4900 4550 4900 4575
+Wire Wire Line
+	4775 4775 5075 4775
+Connection ~ 4900 4775
+Wire Wire Line
+	5275 4775 5600 4775
 $Comp
-L +3.3V #PWR05
-U 1 1 62AF1334
-P 3700 2450
-F 0 "#PWR05" H 3700 2300 50  0001 C CNN
-F 1 "+3.3V" H 3700 2590 50  0000 C CNN
-F 2 "" H 3700 2450 50  0001 C CNN
-F 3 "" H 3700 2450 50  0001 C CNN
-	1    3700 2450
+L C_Small C304
+U 1 1 63E7CCE6
+P 5600 4875
+F 0 "C304" H 5610 4945 50  0000 L CNN
+F 1 "22uf" H 5610 4795 50  0000 L CNN
+F 2 "Capacitors_SMD:C_0603" H 5600 4875 50  0001 C CNN
+F 3 "" H 5600 4875 50  0001 C CNN
+F 4 "603-CC0603MRX6S5B226" H 5600 4875 60  0001 C CNN "Mouser Part Number"
+	1    5600 4875
 	1    0    0    -1
 $EndComp
-$Comp
-L D_Schottky D3
-U 1 1 6303D33A
-P 6100 2500
-F 0 "D3" H 6100 2600 50  0000 C CNN
-F 1 "DFLS240-7" H 6100 2400 50  0000 C CNN
-F 2 "Diodes_SMD:D_PowerDI-123" H 6100 2500 50  0001 C CNN
-F 3 "" H 6100 2500 50  0001 C CNN
-F 4 "621-DFLS240-7" H 6100 2500 60  0001 C CNN "Mouser Part Number"
-	1    6100 2500
-	1    0    0    -1
-$EndComp
+Connection ~ 5375 4775
 Wire Wire Line
-	5950 2500 5950 2750
+	5600 4775 5600 4700
+Wire Wire Line
+	3875 5225 5375 5225
+Wire Wire Line
+	3875 5225 3875 5000
+Wire Wire Line
+	3875 5000 3600 5000
+Connection ~ 3600 5000
+Wire Wire Line
+	5275 4950 4775 4950
+Wire Wire Line
+	5275 4950 5275 4775
+Wire Wire Line
+	5600 4975 5375 4975
+Wire Wire Line
+	5375 4975 5375 5225
+Connection ~ 4275 5225
 $EndSCHEMATC
