File: ESP32-Mini32-OctalServo/MCU.sch (KiCad schematic (older format))
At the start: 1 part, among them U201 TTGO-T7_S3-V1.1

Commit message: Updates to ESP32-Mini32-OctalServo.
Parts:
- U201: symbol TTGO-T7_S3-V1.1 -> TTGO-T7_S3-V1.1-RESCUE-ESP32-Mini32-OctalServo
Changed lines of the file:
@@
 EESchema Schematic File Version 2
+LIBS:ESP32-Mini32-OctalServo-rescue
 LIBS:power
 LIBS:device
@@
 $EndDescr
 $Comp
-L TTGO-T7_S3-V1.1 U201
+L TTGO-T7_S3-V1.1-RESCUE-ESP32-Mini32-OctalServo U201
 U 1 1 63E3CC09
 P 5225 3075
