File: ESP32-Mini32-OctalServo/ESP32-Mini32-OctalServo.sch (KiCad schematic (older format))
At the start: 13 parts, among them J101 + 5V Servo -, J102 Servo 1, J103 Servo 2, J104 Servo 3, J105 Servo 4, J106 Servo 5, J107 Servo 6, J108 Servo 7, J109 Servo 8, U101 74LV125AN, U102 74LV125AN

Commit message: Rescue schematics
Parts:
- U101, U102: symbol 74LV125AN -> 74LV125AN-RESCUE-ESP32-Mini32-OctalServo
Changed lines of the file:
@@
 $EndComp
 $Comp
-L 74LV125AN U101
+L 74LV125AN-RESCUE-ESP32-Mini32-OctalServo U101
 U 1 1 63E3C083
 P 7275 3000
@@
 $EndComp
 $Comp
-L 74LV125AN U101
+L 74LV125AN-RESCUE-ESP32-Mini32-OctalServo U101
 U 3 1 63E3C084
 P 7275 3975
@@
 $EndComp
 $Comp
-L 74LV125AN U101
+L 74LV125AN-RESCUE-ESP32-Mini32-OctalServo U101
 U 2 1 63E3C085
 P 7275 3500
@@
 $EndComp
 $Comp
-L 74LV125AN U101
+L 74LV125AN-RESCUE-ESP32-Mini32-OctalServo U101
 U 4 1 63E3C086
 P 7275 4375
@@
 $EndComp
 $Comp
-L 74LV125AN U102
+L 74LV125AN-RESCUE-ESP32-Mini32-OctalServo U102
 U 1 1 63E3C089
 P 7275 4750
@@
 $EndComp
 $Comp
-L 74LV125AN U102
+L 74LV125AN-RESCUE-ESP32-Mini32-OctalServo U102
 U 3 1 63E3C08A
 P 7300 5625
@@
 $EndComp
 $Comp
-L 74LV125AN U102
+L 74LV125AN-RESCUE-ESP32-Mini32-OctalServo U102
 U 2 1 63E3C08B
 P 7275 5200
@@
 $EndComp
 $Comp
-L 74LV125AN U102
+L 74LV125AN-RESCUE-ESP32-Mini32-OctalServo U102
 U 4 1 63E3C08C
 P 7300 6050
