File: ESP32-T7S3-MultiFunctionUniversalTurnout/OccDetect4.sch (KiCad schematic (older format))
At the start: 35 parts, among them U601 LM339, U602 LM339

Commit message: Minor updates to ESP32-T7S3-MultiFunctionUniversalTurnout.
Parts:
- C601, C602, C603, C604: value 2.2uf 50V -> 2.2uf 35V; Mouser Part Number 710-865080140002 -> 667-EEE-1VA2R2NR
Changed lines of the file:
@@
 $Descr USLetter 11000 8500
 encoding utf-8
-Sheet 6 8
+Sheet 6 7
 Title "ESP32 S3 Multifunction Board"
 Date ""
@@
 P 3850 2050
 F 0 "C601" H 3860 2120 50  0000 L CNN
-F 1 "2.2uf 50V" H 3860 1970 50  0000 L CNN
+F 1 "2.2uf 35V" H 3860 1970 50  0000 L CNN
 F 2 "Capacitors_SMD:CP_Elec_4x5.7" H 3850 2050 50  0001 C CNN
 F 3 "" H 3850 2050 50  0001 C CNN
-F 4 "710-865080140002" H 3850 2050 60  0001 C CNN "Mouser Part Number"
+F 4 "667-EEE-1VA2R2NR" H 3850 2050 60  0001 C CNN "Mouser Part Number"
 	1    3850 2050
 	1    0    0    -1
@@
 P 3850 3250
 F 0 "C602" H 3860 3320 50  0000 L CNN
-F 1 "2.2uf 50V" H 3860 3170 50  0000 L CNN
+F 1 "2.2uf 35V" H 3860 3170 50  0000 L CNN
 F 2 "Capacitors_SMD:CP_Elec_4x5.7" H 3850 3250 50  0001 C CNN
 F 3 "" H 3850 3250 50  0001 C CNN
-F 4 "710-865080140002" H 3850 3250 60  0001 C CNN "Mouser Part Number"
+F 4 "667-EEE-1VA2R2NR" H 3850 3250 60  0001 C CNN "Mouser Part Number"
 	1    3850 3250
 	1    0    0    -1
@@
 P 3850 4550
 F 0 "C603" H 3860 4620 50  0000 L CNN
-F 1 "2.2uf 50V" H 3860 4470 50  0000 L CNN
+F 1 "2.2uf 35V" H 3860 4470 50  0000 L CNN
 F 2 "Capacitors_SMD:CP_Elec_4x5.7" H 3850 4550 50  0001 C CNN
 F 3 "" H 3850 4550 50  0001 C CNN
-F 4 "710-865080140002" H 3850 4550 60  0001 C CNN "Mouser Part Number"
+F 4 "667-EEE-1VA2R2NR" H 3850 4550 60  0001 C CNN "Mouser Part Number"
 	1    3850 4550
 	1    0    0    -1
@@
 P 3850 5950
 F 0 "C604" H 3860 6020 50  0000 L CNN
-F 1 "2.2uf 50V" H 3860 5870 50  0000 L CNN
+F 1 "2.2uf 35V" H 3860 5870 50  0000 L CNN
 F 2 "Capacitors_SMD:CP_Elec_4x5.7" H 3850 5950 50  0001 C CNN
 F 3 "" H 3850 5950 50  0001 C CNN
-F 4 "710-865080140002" H 3850 5950 60  0001 C CNN "Mouser Part Number"
+F 4 "667-EEE-1VA2R2NR" H 3850 5950 60  0001 C CNN "Mouser Part Number"
 	1    3850 5950
 	1    0    0    -1
