File: ESP32-T7S3-MultiFunctionUniversalTurnout/CAN_Transceiver.kicad_sch (KiCad schematic)
At the start: 13 parts, among them J801 RJ45, J802 RJ45, T801 - 15 in +, T802 - 15 out +, U801 TCAN332DR

Commit message: Update part numbers.
Parts:
- C802: Mouser Part Number 647-UUD1C150MCL -> 710-865080340002
Changed lines of the file:
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@@
       (effects (font (size 1.524 1.524)))
     )
-    (property "Mouser Part Number" "647-UUD1C150MCL" (id 4) (at 127 96.52 0)
+    (property "Mouser Part Number" "710-865080340002 " (id 4) (at 127 96.52 0)
       (effects (font (size 1.524 1.524)) hide)
     )
