File: ESP32-T7S3-MultiFunctionUniversalTurnout/PowerSupply.kicad_sch (KiCad schematic)
At the start: 6 parts, among them U301 AP63205

Commit message: Update part numbers.
Parts:
- L301: Mouser Part Number 81-B1047AS-4R7NP3 -> 81-B1047AS-4R7N=P3
Changed lines of the file:
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@@
       (effects (font (size 1.27 1.27)) hide)
     )
-    (property "Mouser Part Number" "81-B1047AS-4R7NP3" (id 4) (at 131.445 121.285 0)
+    (property "Mouser Part Number" "81-B1047AS-4R7N=P3" (id 4) (at 131.445 121.285 0)
       (effects (font (size 1.524 1.524)) hide)
     )
