File: ESP32-T7S3-MultiFunctionUniversalTurnout/ESP32-MCU.sch (KiCad schematic (older format))
At the start: 7 parts, among them U201 TTGO-T7_S3-V1.1

Commit message: Fix component part number.
Parts:
- R203, R206: Mouser Part Number 71-CRCW06032K40JNEAC -> 71-RC0402FR-072K4L
Changed lines of the file:
@@
 F 2 "Resistors_SMD:R_0402" V 3980 3750 50  0001 C CNN
 F 3 "" H 4050 3750 50  0001 C CNN
-F 4 "71-CRCW06032K40JNEAC" V 4050 3750 60  0001 C CNN "Mouser Part Number"
+F 4 "71-RC0402FR-072K4L" V 4050 3750 60  0001 C CNN "Mouser Part Number"
 	1    4050 3750
 	1    0    0    -1
@@
 F 2 "Resistors_SMD:R_0402" V 3530 3850 50  0001 C CNN
 F 3 "" H 3600 3850 50  0001 C CNN
-F 4 "71-CRCW06032K40JNEAC" V 3600 3850 60  0001 C CNN "Mouser Part Number"
+F 4 "71-RC0402FR-072K4L" V 3600 3850 60  0001 C CNN "Mouser Part Number"
 	1    3600 3850
 	-1   0    0    1
