File: ESP32-Mini32-OctalBuffer/MCU.sch (KiCad schematic (older format))
At the start: 1 part, among them U201 TTGO-T7_S3-V1.1

Commit message: Rescue T7 S3
Parts:
- U201: symbol TTGO-T7_S3-V1.1 -> TTGO-T7_S3-V1.1-RESCUE-ESP32-Mini32-OctalBuffer
Changed lines of the file:
@@
 EESchema Schematic File Version 2
+LIBS:ESP32-Mini32-OctalBuffer-rescue
 LIBS:power
 LIBS:device
@@
 $EndDescr
 $Comp
-L TTGO-T7_S3-V1.1 U201
+L TTGO-T7_S3-V1.1-RESCUE-ESP32-Mini32-OctalBuffer U201
 U 1 1 63E00230
 P 5225 3075
