File: ESP32-Mini32-OctalBuffer/MCU.kicad_sch (KiCad schematic)
At the start: 1 part, among them U201 TTGO-T7_S3-V1.1

Commit message: Add LCSC Part numbers.
Parts:
- U201: now left out of the parts list
Changed lines of the file:
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@@
   )
   (symbol (lib_id "ESP32-Mini32-OctalBuffer-rescue:TTGO-T7_S3-V1.1-RESCUE-ESP32-Mini32-OctalBuffer") (at 132.715 78.105 0) (unit 1)
-    (in_bom yes) (on_board yes)
+    (in_bom no) (on_board yes)
     (property "Reference" "U201" (id 0) (at 139.7 127.635 0))
     (property "Value" "TTGO-T7_S3-V1.1" (id 1) (at 135.255 146.05 0))
@@
     (pin "1")
   )
-  (symbol (lib_id "ESP32-Mini32-OctalBuffer-rescue:+3V3") (at 152.4 83.185 0)
+  (symbol (lib_id "ESP32-Mini32-OctalBuffer-rescue:+3V3") (at 152.4 83.185 0) (unit 1)
     (in_bom yes) (on_board yes)
     (property "Reference" "#PWR05" (id 0) (at 152.4 86.995 0)
