File: ESP32-T7S3-TextDisplaySign/DisplayBoard.kicad_sch (KiCad schematic)
At the start: 3 parts

Commit message: Complete draft board layout.
Parts:
- J501: renamed from J?; value G K A RST RS D C CS1 CS2 Vcc -> Vcc CS2 CS1 C D RS RST A K G; footprint (none) -> Connector_PinHeader_2.54mm:PinHeader_1x10_P2.54mm_Horizontal
- gave numbers to parts that had none: 2
Connections:
- net +3V3: now reaches J501.10 (Pin_10), LCD501.10 (Vcc), LCD501.11 (Vcc), LCD502.10 (Vcc), LCD502.11 (Vcc)
- net GND: now reaches J501.1 (Pin_1), LCD501.13 (GND), LCD501.2 (GND), LCD501.5 (GND), LCD502.13 (GND), LCD502.2 (GND), LCD502.5 (GND)
Changed lines of the file:
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@@
   (junction (at 156.845 63.5) (diameter 0) (color 0 0 0 0)
   )
+  (junction (at 131.445 48.26) (diameter 0) (color 0 0 0 0)
+  )
   (junction (at 146.05 53.34) (diameter 0) (color 0 0 0 0)
   )
@@
   (junction (at 147.955 74.295) (diameter 0) (color 0 0 0 0)
   )
+  (junction (at 133.35 91.44) (diameter 0) (color 0 0 0 0)
+  )
   (junction (at 144.145 91.44) (diameter 0) (color 0 0 0 0)
   )
@@
     (stroke (width 0) (type default) (color 0 0 0 0))
   )
-  (wire (pts (xy 139.065 48.26) (xy 128.27 48.26))
+  (wire (pts (xy 139.065 48.26) (xy 131.445 48.26))
     (stroke (width 0) (type default) (color 0 0 0 0))
   )
@@
     (stroke (width 0) (type default) (color 0 0 0 0))
   )
+  (wire (pts (xy 133.35 91.44) (xy 128.27 91.44))
+    (stroke (width 0) (type default) (color 0 0 0 0))
+  )
   (wire (pts (xy 144.145 52.07) (xy 161.925 52.07))
     (stroke (width 0) (type default) (color 0 0 0 0))
@@
     (stroke (width 0) (type default) (color 0 0 0 0))
   )
-  (wire (pts (xy 144.145 91.44) (xy 128.27 91.44))
+  (wire (pts (xy 144.145 91.44) (xy 133.35 91.44))
     (stroke (width 0) (type default) (color 0 0 0 0))
   )
@@
   (wire (pts (xy 146.05 78.105) (xy 160.655 78.105))
     (stroke (width 0) (type default) (color 0 0 0 0))
+  )
+  (wire (pts (xy 131.445 48.26) (xy 128.27 48.26))
+    (stroke (width 0) (type default) (color 0 0 0 0))
+  )
+  (symbol (lib_id "ESP32-T7S3-MultiFunctionUniversalTurnout-rescue:GND") (at 131.445 48.26 0) (unit 1)
+    (in_bom yes) (on_board yes) (fields_autoplaced)
+    (property "Reference" "#PWR?" (id 0) (at 131.445 54.61 0)
+      (effects (font (size 1.27 1.27)) hide)
+    )
+    (property "Value" "GND" (id 1) (at 131.445 53.34 0))
+    (property "Footprint" "" (id 2) (at 131.445 48.26 0)
+      (effects (font (size 1.27 1.27)) hide)
+    )
+    (property "Datasheet" "" (id 3) (at 131.445 48.26 0)
+      (effects (font (size 1.27 1.27)) hide)
+    )
+    (pin "1")
+  )
+  (symbol (lib_id "ESP32-T7S3-MultiFunctionUniversalTurnout-rescue:+3V3") (at 133.35 91.44 0) (unit 1)
+    (in_bom yes) (on_board yes) (fields_autoplaced)
+    (property "Reference" "#PWR?" (id 0) (at 133.35 95.25 0)
+      (effects (font (size 1.27 1.27)) hide)
+    )
+    (property "Value" "+3V3" (id 1) (at 133.35 86.36 0))
+    (property "Footprint" "" (id 2) (at 133.35 91.44 0)
+      (effects (font (size 1.27 1.27)) hide)
+    )
+    (property "Datasheet" "" (id 3) (at 133.35 91.44 0)
+      (effects (font (size 1.27 1.27)) hide)
+    )
+    (pin "1")
   )
   (symbol (lib_id "JD-T1800:JD-T1800") (at 183.515 86.36 0) (unit 1)
     (in_bom yes) (on_board yes) (fields_autoplaced)
-    (property "Reference" "LCD?" (id 0) (at 202.565 86.3599 0)
+    (property "Reference" "LCD501" (id 0) (at 202.565 86.3599 0)
       (effects (font (size 1.27 1.27)) (justify left))
     )
@@
   (symbol (lib_id "JD-T1800:JD-T1800") (at 184.785 46.99 0) (unit 1)
     (in_bom yes) (on_board yes) (fields_autoplaced)
-    (property "Reference" "LCD?" (id 0) (at 203.835 46.9899 0)
+    (property "Reference" "LCD502" (id 0) (at 203.835 46.9899 0)
       (effects (font (size 1.27 1.27)) (justify left))
     )
@@
   (symbol (lib_id "Connector:Conn_01x10_Male") (at 123.19 58.42 0) (unit 1)
     (in_bom yes) (on_board yes)
-    (property "Reference" "J?" (id 0) (at 124.46 45.72 0))
-    (property "Value" "G K A RST RS D C CS1 CS2 Vcc" (id 1) (at 118.745 58.42 90))
-    (property "Footprint" "" (id 2) (at 123.19 58.42 0)
-      (effects (font (size 1.27 1.27)) hide)
-    )
+    (property "Reference" "J501" (id 0) (at 124.46 45.72 0))
+    (property "Value" "Vcc CS2 CS1 C D RS RST A K G" (id 1) (at 118.745 58.42 90))
+    (property "Footprint" "Connector_PinHeader_2.54mm:PinHeader_1x10_P2.54mm_Horizontal" (id 2) (at 123.19 58.42 0)
+      (effects (font (size 1.27 1.27)) hide)
+    )

Commit message: Board dims and part numbers for BOM.
Parts:
- LCD501: Manufacturer_Name (none) -> Jiandakangjing Technology, Co., Ltd.; Manufacturer_Part_Number (none) -> JD-T18002-T01
- LCD502: Manufacturer_Name (none) -> Jiandakangjing Technology, Co., Ltd.; Manufacturer_Part_Number_index (none) -> JD-T18002-T01
Changed lines of the file:
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@@
   (symbol (lib_id "ESP32-T7S3-MultiFunctionUniversalTurnout-rescue:GND") (at 131.445 48.26 0) (unit 1)
     (in_bom yes) (on_board yes) (fields_autoplaced)
-    (property "Reference" "#PWR?" (id 0) (at 131.445 54.61 0)
+    (property "Reference" "#PWR0108" (id 0) (at 131.445 54.61 0)
       (effects (font (size 1.27 1.27)) hide)
     )
@@
   (symbol (lib_id "ESP32-T7S3-MultiFunctionUniversalTurnout-rescue:+3V3") (at 133.35 91.44 0) (unit 1)
     (in_bom yes) (on_board yes) (fields_autoplaced)
-    (property "Reference" "#PWR?" (id 0) (at 133.35 95.25 0)
+    (property "Reference" "#PWR0109" (id 0) (at 133.35 95.25 0)
       (effects (font (size 1.27 1.27)) hide)
     )
@@
     )
     (property "Datasheet" "" (id 3) (at 183.515 86.36 0)
+      (effects (font (size 1.27 1.27)) hide)
+    )
+    (property "Manufacturer_Name" "Jiandakangjing Technology, Co., Ltd." (id 4) (at 183.515 86.36 0)
+      (effects (font (size 1.27 1.27)) hide)
+    )
+    (property "Manufacturer_Part_Number" "JD-T18002-T01" (id 5) (at 183.515 86.36 0)
       (effects (font (size 1.27 1.27)) hide)
     )
@@
       (effects (font (size 1.27 1.27)) hide)
     )
+    (property "Manufacturer_Name" "Jiandakangjing Technology, Co., Ltd." (id 4) (at 184.785 46.99 0)
+      (effects (font (size 1.27 1.27)) hide)
+    )
+    (property "Manufacturer_Part_Number_index" "JD-T18002-T01" (id 5) (at 184.785 46.99 0)
+      (effects (font (size 1.27 1.27)) hide)
+    )
