File: ESP32-T7S3-TextDisplaySign/ESP32-T7S3-TextDisplaySign.kicad_sch (KiCad schematic)
At the start: 5 parts

Commit message: ESP32-T7S3-TextDisplaySign.
Other:
- sheet Processor ports: added Backlight , CardCS, DCS1, DCS2, DReset, DRs, MISO, MOSI, SCLK; removed none
Changed lines of the file:
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@@
     (effects (font (size 1.27 1.27)) (justify right bottom))
+  )
+  (label "MOSI" (at 159.385 64.135 0)
+    (effects (font (size 1.27 1.27)) (justify left bottom))
   )
   (label "DRS" (at 193.04 53.975 0)
@@
     (effects (font (size 1.27 1.27)) (justify right bottom))
   )
+  (label "CardCS" (at 159.385 60.325 0)
+    (effects (font (size 1.27 1.27)) (justify left bottom))
+  )
+  (label "DReset" (at 159.385 52.705 0)
+    (effects (font (size 1.27 1.27)) (justify left bottom))
+  )
+  (label "SCLK" (at 159.385 66.04 0)
+    (effects (font (size 1.27 1.27)) (justify left bottom))
+  )
   (label "DCS2" (at 180.34 61.595 180)
     (effects (font (size 1.27 1.27)) (justify right bottom))
@@
     (effects (font (size 1.27 1.27)) (justify left bottom))
   )
+  (label "DRS" (at 159.385 54.61 0)
+    (effects (font (size 1.27 1.27)) (justify left bottom))
+  )
   (label "MISO" (at 203.835 110.49 180)
     (effects (font (size 1.27 1.27)) (justify right bottom))
@@
     (effects (font (size 1.27 1.27)) (justify left bottom))
   )
+  (label "MISO" (at 159.385 62.23 0)
+    (effects (font (size 1.27 1.27)) (justify left bottom))
+  )
   (label "DA" (at 180.34 53.975 180)
     (effects (font (size 1.27 1.27)) (justify right bottom))
@@
     (effects (font (size 1.27 1.27)) (justify left bottom))
   )
+  (label "DCS2" (at 159.385 58.42 0)
+    (effects (font (size 1.27 1.27)) (justify left bottom))
+  )
   (label "CardCS" (at 203.835 97.79 180)
     (effects (font (size 1.27 1.27)) (justify right bottom))
   )
+  (label "Backlight" (at 159.385 50.8 0)
+    (effects (font (size 1.27 1.27)) (justify left bottom))
+  )
   (label "DReset" (at 180.34 56.515 180)
     (effects (font (size 1.27 1.27)) (justify right bottom))
+  )
+  (label "DCS1" (at 159.385 56.515 0)
+    (effects (font (size 1.27 1.27)) (justify left bottom))
   )
   (label "MOSI" (at 203.835 100.33 180)
@@
       (effects (font (size 1.27 1.27)) (justify left))
     )
-  )
+    (pin "MOSI" output (at 159.385 64.135 0)
+      (effects (font (size 1.27 1.27)) (justify right))
+    )
+    (pin "SCLK" output (at 159.385 66.04 0)
+      (effects (font (size 1.27 1.27)) (justify right))
+    )
+    (pin "MISO" input (at 159.385 62.23 0)
+      (effects (font (size 1.27 1.27)) (justify right))
+    )
+    (pin "Backlight " output (at 159.385 50.8 0)
+      (effects (font (size 1.27 1.27)) (justify right))
+    )
+    (pin "DReset" output (at 159.385 52.705 0)
+      (effects (font (size 1.27 1.27)) (justify right))
+    )
+    (pin "DRs" output (at 159.385 54.61 0)
+      (effects (font (size 1.27 1.27)) (justify right))
+    )
+    (pin "DCS1" output (at 159.385 56.515 0)
+      (effects (font (size 1.27 1.27)) (justify right))
+    )
+    (pin "DCS2" output (at 159.385 58.42 0)
+      (effects (font (size 1.27 1.27)) (justify right))
+    )
+    (pin "CardCS" output (at 159.385 60.325 0)
+      (effects (font (size 1.27 1.27)) (justify right))
+    )
+  )

Commit message: Complete draft board layout.
Parts:
- J102: renamed from J?; footprint (none) -> Connector_Card:microSD_HC_Hirose_DM3D-SF; Mouser Part Number (none) -> 798-DM3D-SF
- gave numbers to parts that had none: 4

Commit message: Board dims and part numbers for BOM.
Parts:
- Q101: Mouser Part Number (none) -> 771-PZT2222A135
- R101: Mouser Part Number (none) -> 603-RT0603DRE0722RL
- R102: Mouser Part Number (none) -> 603-AC0402JR-7D1KL
Changed lines of the file:
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@@
+      (effects (font (size 1.27 1.27)) hide)
+    )
+    (property "Mouser Part Number" "603-AC0402JR-7D1KL" (id 4) (at 215.9 33.655 90)
       (effects (font (size 1.27 1.27)) hide)
     )
@@
     )
     (property "Datasheet" "~" (id 3) (at 200.66 44.45 0)
+      (effects (font (size 1.27 1.27)) hide)
+    )
+    (property "Mouser Part Number" "603-RT0603DRE0722RL" (id 4) (at 200.66 44.45 0)
       (effects (font (size 1.27 1.27)) hide)
     )
@@
       (effects (font (size 1.27 1.27)) (justify left) hide)
     )
+    (property "Mouser Part Number" "771-PZT2222A135" (id 4) (at 203.2 33.655 0)
+      (effects (font (size 1.27 1.27)) hide)
+    )
     (pin "1")
     (pin "2")
@@
     )
     (path "/0dbdf17a-1f86-4bad-b68c-59be1dcdeafb/1321877b-b430-490c-b8ff-14bc5d133a03"
-      (reference "#PWR?") (unit 1) (value "GND") (footprint "")
+      (reference "#PWR0108") (unit 1) (value "GND") (footprint "")
     )
     (path "/0dbdf17a-1f86-4bad-b68c-59be1dcdeafb/6f1c8c53-1945-4ded-bc8c-09b24922f02a"
-      (reference "#PWR?") (unit 1) (value "+3V3") (footprint "")
+      (reference "#PWR0109") (unit 1) (value "+3V3") (footprint "")
     )
     (path "/58a06321-5405-479d-b5db-3c7330a446c5/00000000-0000-0000-0000-000063e7cce1"
