File: ESP32-Feather-6B6L/6Buttons.kicad_sch (KiCad schematic)
At the start: 15 parts, among them J401 1 2 3 4 5 6 G, U403 74HCT14

Commit message: Final through-hole tweaks.
Parts:
- J401: value 1 2 3 4 5 6 G -> G 6 5 4 3 2 1
Changed lines of the file:
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@@
     (in_bom yes) (on_board yes)
     (property "Reference" "J401" (id 0) (at 164.465 62.23 0))
-    (property "Value" "1 2 3 4 5 6 G" (id 1) (at 159.385 76.2 90))
+    (property "Value" "G  6  5  4  3  2  1" (id 1) (at 159.385 76.2 90))
     (property "Footprint" "TerminalBlock_TE-Connectivity:TerminalBlock_TE_282834-7_1x07_P2.54mm_Horizontal" (id 2) (at 164.465 76.2 0)
       (effects (font (size 1.27 1.27)) hide)
