File: T7S3-MiniDisplay/PowerSupply.kicad_sch (KiCad schematic)
At the start: 6 parts, among them U301 AP63205

Commit message: Finalize part numbers.
Parts:
- C301: MPN (none) -> EEE-HB1C100R; Mouser Part Number 710-865230542002 -> 667-EEE-HB1C100R
- C302: MPN (none) -> 885012206020
- C303, C304: MPN (none) -> CC0603MRX6S5B226
- L301: MPN (none) -> B1047AS-4R7N=P3
- U301: MPN (none) -> AP63205WU-7
Changed lines of the file:
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@@
       (effects (font (size 1.524 1.524)) hide)
+    )
+    (property "MPN" "AP63205WU-7" (id 5) (at 108.585 121.285 0)
+      (effects (font (size 1.27 1.27)) hide)
     )
     (pin "1")
@@
       (effects (font (size 1.27 1.27)) hide)
     )
-    (property "Mouser Part Number" "710-865230542002" (id 4) (at 91.44 121.92 0)
+    (property "Mouser Part Number" "667-EEE-HB1C100R" (id 4) (at 91.44 121.92 0)
       (effects (font (size 1.524 1.524)) hide)
+    )
+    (property "MPN" "EEE-HB1C100R" (id 5) (at 91.44 121.92 0)
+      (effects (font (size 1.27 1.27)) hide)
     )
     (pin "1")
@@
       (effects (font (size 1.524 1.524)) hide)
     )
+    (property "MPN" "885012206020" (id 5) (at 124.46 118.745 0)
+      (effects (font (size 1.27 1.27)) hide)
+    )
     (pin "1")
     (pin "2")
@@
     (property "Mouser Part Number" "81-B1047AS-4R7N=P3" (id 4) (at 131.445 121.285 0)
       (effects (font (size 1.524 1.524)) hide)
+    )
+    (property "MPN" "B1047AS-4R7N=P3" (id 5) (at 131.445 121.285 0)
+      (effects (font (size 1.27 1.27)) hide)
     )
     (pin "1")
@@
       (effects (font (size 1.524 1.524)) hide)
     )
+    (property "MPN" "CC0603MRX6S5B226" (id 5) (at 136.525 123.825 0)
+      (effects (font (size 1.27 1.27)) hide)
+    )
     (pin "1")
     (pin "2")
@@
       (effects (font (size 1.524 1.524)) hide)
     )
+    (property "MPN" "CC0603MRX6S5B226" (id 5) (at 142.24 123.825 0)
+      (effects (font (size 1.27 1.27)) hide)
+    )
     (pin "1")
