File: T7S3-MiniDisplay/T7S3-MiniDisplay.kicad_sch (KiCad schematic)
At the start: 11 parts, among them J101 Qwicc, J102 Micro_SD_Card_Det, U101 TTGO-T7_S3-V1.1

Commit message: Finalize part numbers.
Parts:
- C101: MPN (none) -> EEE-HB1C100R; Mouser Part Number  710-865080340001 -> 667-EEE-HB1C100R
- C102: MPN (none) -> C0603C104K5RAC7411; Mouser Part Number 710-885012206095 -> 80-C0603C104K5R7411
- H101, H102, H103, U101: now left out of the parts list
- J101: footprint Connector_JST:JST_SH_SM04B-SRSS-TB_1x04-1MP_P1.00mm_Horizontal -> Connector_JST:JST_PH_S4B-PH-SM4-TB_1x04-1MP_P2.00mm_Horizontal; MPN (none) -> S4B-PH-SM4-TB(LF)(SN); Manufacturer (none) -> JST; Mouser Part Number (none) -> 306-S4BPHSM4TBLFSN
- R101, R102: MPN (none) -> RE0603DRE0710KL; Manufacturer Part Number RE0603DRE0710KL -> (none)
- R103: MPN (none) -> YC158TJR-0747KL; Manufacturer Part Number YC158TJR-0747KL -> (none)
Changed lines of the file:
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@@
       (effects (font (size 1.27 1.27)) hide)
     )
-    (property "Mouser Part Number" "710-885012206095" (id 4) (at 158.75 118.745 0)
+    (property "Mouser Part Number" "80-C0603C104K5R7411" (id 4) (at 158.75 118.745 0)
+      (effects (font (size 1.27 1.27)) hide)
+    )
+    (property "MPN" "C0603C104K5RAC7411" (id 5) (at 158.75 118.745 0)
       (effects (font (size 1.27 1.27)) hide)
     )
@@
   )
   (symbol (lib_id "ESP32_mini:TTGO-T7_S3-V1.1") (at 119.38 36.83 0) (unit 1)
-    (in_bom yes) (on_board yes) (fields_autoplaced)
+    (in_bom no) (on_board yes) (fields_autoplaced)
     (property "Reference" "U101" (id 0) (at 120.015 33.02 0))
     (property "Value" "TTGO-T7_S3-V1.1" (id 1) (at 120.015 35.56 0))
@@
   )
   (symbol (lib_id "Mechanical:MountingHole") (at 98.425 153.035 0) (unit 1)
-    (in_bom yes) (on_board yes) (fields_autoplaced)
+    (in_bom no) (on_board yes) (fields_autoplaced)
     (property "Reference" "H103" (id 0) (at 100.965 151.7649 0)
       (effects (font (size 1.27 1.27)) (justify left) hide)
@@
       (effects (font (size 1.27 1.27)) hide)
     )
-    (property "Manufacturer Part Number" "RE0603DRE0710KL" (id 6) (at 73.66 107.95 0)
+    (property "MPN" "RE0603DRE0710KL" (id 6) (at 73.66 107.95 0)
       (effects (font (size 1.27 1.27)) hide)
     )
@@
   )
   (symbol (lib_id "Mechanical:MountingHole") (at 87.63 153.035 0) (unit 1)
-    (in_bom yes) (on_board yes) (fields_autoplaced)
+    (in_bom no) (on_board yes) (fields_autoplaced)
     (property "Reference" "H101" (id 0) (at 90.17 151.7649 0)
       (effects (font (size 1.27 1.27)) (justify left) hide)
@@
   )
   (symbol (lib_id "Mechanical:MountingHole") (at 93.345 153.67 0) (unit 1)
-    (in_bom yes) (on_board yes) (fields_autoplaced)
+    (in_bom no) (on_board yes) (fields_autoplaced)
     (property "Reference" "H102" (id 0) (at 95.885 152.3999 0)
       (effects (font (size 1.27 1.27)) (justify left) hide)
@@
       (effects (font (size 1.27 1.27)) hide)
     )
-    (property "Manufacturer Part Number" "RE0603DRE0710KL" (id 6) (at 76.835 107.95 0)
+    (property "MPN" "RE0603DRE0710KL" (id 6) (at 76.835 107.95 0)
       (effects (font (size 1.27 1.27)) hide)
     )
@@
       (effects (font (size 1.27 1.27)) hide)
     )
-    (property "Mouser Part Number " "710-865080340001" (id 4) (at 150.495 118.745 0)
+    (property "Mouser Part Number " "667-EEE-HB1C100R" (id 4) (at 150.495 118.745 0)
+      (effects (font (size 1.27 1.27)) hide)
+    )
+    (property "MPN" "EEE-HB1C100R" (id 5) (at 150.495 118.745 0)
       (effects (font (size 1.27 1.27)) hide)
     )
@@
       (effects (font (size 1.27 1.27)) (justify left top) hide)
     )
-    (property "Manufacturer Part Number" "YC158TJR-0747KL" (id 12) (at 168.275 888.9 0)
+    (property "MPN" "YC158TJR-0747KL" (id 12) (at 168.275 888.9 0)
       (effects (font (size 1.27 1.27)) (justify left top) hide)
     )
@@
     (property "Reference" "J101" (id 0) (at 64.135 105.41 0))
     (property "Value" "Qwicc" (id 1) (at 64.135 107.95 0))
-    (property "Footprint" "Connector_JST:JST_SH_SM04B-SRSS-TB_1x04-1MP_P1.00mm_Horizontal" (id 2) (at 63.5 113.665 0)
+    (property "Footprint" "Connector_JST:JST_PH_S4B-PH-SM4-TB_1x04-1MP_P2.00mm_Horizontal" (id 2) (at 63.5 113.665 0)
       (effects (font (size 1.27 1.27)) hide)
     )
     (property "Datasheet" "~" (id 3) (at 63.5 113.665 0)
+      (effects (font (size 1.27 1.27)) hide)
+    )
+    (property "MPN" "S4B-PH-SM4-TB(LF)(SN) " (id 4) (at 63.5 113.665 0)
+      (effects (font (size 1.27 1.27)) hide)
+    )
+    (property "Mouser Part Number" "306-S4BPHSM4TBLFSN " (id 5) (at 63.5 113.665 0)
+      (effects (font (size 1.27 1.27)) hide)
+    )
+    (property "Manufacturer" "JST" (id 6) (at 63.5 113.665 0)
       (effects (font (size 1.27 1.27)) hide)
     )
@@
     )
     (path "/e1161042-1605-4ce0-8903-857b3bfb0710"
-      (reference "J101") (unit 1) (value "Qwicc") (footprint "Connector_JST:JST_SH_SM04B-SRSS-TB_1x04-1MP_P1.00mm_Horizontal")
+      (reference "J101") (unit 1) (value "Qwicc") (footprint "Connector_JST:JST_PH_S4B-PH-SM4-TB_1x04-1MP_P2.00mm_Horizontal")
     )
     (path "/5b1ec8bd-43ed-4157-b754-1075ffa0e621"
