File: P9WiFiLCCTraction_Sound/P9WiFiLCCTraction_Sound.kicad_sch (KiCad schematic)
At the start: 31 parts, among them IC102 MP6614GN-Z, J101 USB_C_Receptacle, J102 DCC 9-pin, SW101 Reset, SW102 Boot, U101 ESP32_S3_WROOM, U102 TBD62064AFG_1, U103 AP63203WU

Commit message: Complete P9WiFiLCCTraction_Sound hardware.
Parts:
- added C111: .1uf, Capacitor_SMD:C_0402_1005Metric, symbol Device:C
- added C112: 10uf 6.3V, Capacitor_SMD:C_0603_1608Metric, symbol Device:C
- added R104: 0, Resistor_SMD:R_0402_1005Metric, symbol Device:R
- added TP101: Speaker, TestPoint:TestPoint_2Pads_Pitch2.54mm_Drill0.8mm, symbol Connector:TestPoint_2Pole
- added U104: MAX98357AETE+T, Package_DFN_QFN:TQFN-16-1EP_3x3mm_P0.5mm_EP1.23x1.23mm_ThermalVias, symbol MAX98357A:MAX98357AETE+T
Connections:
- net +3V3: now also C111.1, C112.1, R104.1, U104.7 (VDD_1), U104.8 (VDD_2)
- net GND: now also C111.2, C112.2, U104.11 (GND_2), U104.15 (GND_3), U104.17 (THERMAL_PAD), U104.2 (GAIN_SLOT), U104.3 (GND_1)
- net I2S_TX: now reaches U101.19 (IO11)
- net I2S_TX: now also U104.1 (DIN)
- net I2S_BCLK: now reaches U101.20 (IO12)
- net I2S_BCLK: now also U104.16 (BCLK)
- net LRCLK: now reaches U101.21 (IO13)
- net LRCLK: now also U104.14 (LRCLK)
- new net: TP101.2, U104.10 (OUTN)
- new net: R104.2, U104.4 (~{SD_MODE})
- new net: TP101.1, U104.9 (OUTP)
- no-connect marks 38 -> 39
Other:
- moved on the sheet: C103, C104, C105, J102, R103, R105, R106, R107, SW102, TP104, U102A, U102B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

Commit message: Final (silkscreen) tweaks, Image files generated.
Other:
- title: JST 9-Pin WiFi LCC Traction Node -> JST 9-Pin WiFi LCC Traction Node w/ Sound
Changed lines of the file:
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@@
   (paper "USLetter")
   (title_block
-    (title "JST 9-Pin WiFi LCC Traction Node")
+    (title "JST 9-Pin WiFi LCC Traction Node w/ Sound")
     (date "12/11/2025")
     (rev "A")
