File: AdafruitMetroESP32-S3-CANLCC-Shield/AdafruitMetroESP32-S3-CANLCC-Shield.kicad_sch (KiCad schematic)
At the start: 33 parts, among them J1 Power, J101 MA MB NA NB, J102 S4 S3 S2 S1 SC, J103 - 12V +, J104 B1 C B2, J105 LCC, J106 LCC, J107 Servo 4, J108 Servo 3, J109 Servo 2, J110 Servo 1, J2 Digital/PWM, J3 Analog, J4 Digital/PWM, U101 TBD62064AFG, U102 TC4428, U103 TC4428, U104 G3VM-61VY4, U105 G3VM-61VY4, U106 LM358, U107 TCAN332DR

Commit message: Snapshot commit -- PCB almost done.
Parts:
- J102: value S4 S3 S2 S1 SC -> S1 S2 S3 S4 SC
- J104: value B1 C B2 -> B2 C B1
- J107: value Servo 4 -> Sv 4
- J108: value Servo 3 -> Sv 3
- J109: value Servo 2 -> Sv 2
- J110: value Servo 1 -> Sv 1
Changed lines of the file:
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@@
     (effects (font (size 1.27 1.27)) (justify left bottom))
   )
-  (label "Motor_A" (at 74.93 62.23 0)
+  (label "Motor_M" (at 74.93 62.23 0)
     (effects (font (size 1.27 1.27)) (justify left bottom))
   )
@@
     (effects (font (size 1.27 1.27)) (justify left bottom))
   )
-  (label "Motor_B" (at 74.93 59.69 0)
+  (label "Motor_N" (at 74.93 59.69 0)
     (effects (font (size 1.27 1.27)) (justify left bottom))
   )
@@
     (effects (font (size 1.27 1.27)) (justify right bottom))
   )
-  (label "Motor_B" (at 133.985 100.33 0)
+  (label "Motor_N" (at 133.985 100.33 0)
     (effects (font (size 1.27 1.27)) (justify left bottom))
   )
@@
     (effects (font (size 1.27 1.27)) (justify right bottom))
   )
-  (label "Motor_A" (at 133.35 139.7 0)
+  (label "Motor_M" (at 133.35 139.7 0)
     (effects (font (size 1.27 1.27)) (justify left bottom))
   )
@@
     (in_bom no) (on_board yes)
     (property "Reference" "J107" (id 0) (at 274.32 25.4 0))
-    (property "Value" "Servo 4" (id 1) (at 274.32 35.56 0))
+    (property "Value" "Sv 4" (id 1) (at 274.32 35.56 0))
     (property "Footprint" "Connector_PinHeader_2.54mm:PinHeader_1x03_P2.54mm_Vertical" (id 2) (at 274.32 30.48 0)
       (effects (font (size 1.27 1.27)) hide)
@@
     (in_bom no) (on_board yes)
     (property "Reference" "J108" (id 0) (at 274.32 36.83 0))
-    (property "Value" "Servo 3" (id 1) (at 274.32 46.99 0))
+    (property "Value" "Sv 3" (id 1) (at 274.32 46.99 0))
     (property "Footprint" "Connector_PinHeader_2.54mm:PinHeader_1x03_P2.54mm_Vertical" (id 2) (at 274.32 41.91 0)
       (effects (font (size 1.27 1.27)) hide)
@@
     (in_bom no) (on_board yes)
     (property "Reference" "J110" (id 0) (at 274.32 55.245 0))
-    (property "Value" "Servo 1" (id 1) (at 274.32 65.405 0))
+    (property "Value" "Sv 1" (id 1) (at 274.32 65.405 0))
     (property "Footprint" "Connector_PinHeader_2.54mm:PinHeader_1x03_P2.54mm_Vertical" (id 2) (at 274.32 60.325 0)
       (effects (font (size 1.27 1.27)) hide)
@@
     (in_bom no) (on_board yes)
     (property "Reference" "J104" (id 0) (at 224.155 29.21 0))
-    (property "Value" "B1 C B2" (id 1) (at 224.155 39.37 0))
+    (property "Value" "B2 C B1" (id 1) (at 224.155 39.37 0))
     (property "Footprint" "TerminalBlock_TE-Connectivity:TerminalBlock_TE_282834-3_1x03_P2.54mm_Horizontal" (id 2) (at 224.155 34.29 0)
       (effects (font (size 1.27 1.27)) hide)
@@
     (in_bom no) (on_board yes)
     (property "Reference" "J109" (id 0) (at 274.32 46.355 0))
-    (property "Value" "Servo 2" (id 1) (at 274.32 56.515 0))
+    (property "Value" "Sv 2" (id 1) (at 274.32 56.515 0))
     (property "Footprint" "Connector_PinHeader_2.54mm:PinHeader_1x03_P2.54mm_Vertical" (id 2) (at 274.32 51.435 0)
       (effects (font (size 1.27 1.27)) hide)
@@
     (in_bom no) (on_board yes)
     (property "Reference" "J102" (id 0) (at 101.6 42.545 0))
-    (property "Value" "S4 S3 S2 S1 SC" (id 1) (at 101.6 57.785 0))
+    (property "Value" "S1 S2 S3 S4 SC" (id 1) (at 101.6 57.785 0))
     (property "Footprint" "TerminalBlock_Phoenix:TerminalBlock_Phoenix_MPT-0,5-5-2.54_1x05_P2.54mm_Horizontal" (id 2) (at 101.6 50.165 0)
       (effects (font (size 1.27 1.27)) hide)
@@
     )
     (path "/fcda36f3-9929-43cd-b355-545a49abf1e2"
-      (reference "J102") (unit 1) (value "S4 S3 S2 S1 SC") (footprint "TerminalBlock_Phoenix:TerminalBlock_Phoenix_MPT-0,5-5-2.54_1x05_P2.54mm_Horizontal")
+      (reference "J102") (unit 1) (value "S1 S2 S3 S4 SC") (footprint "TerminalBlock_Phoenix:TerminalBlock_Phoenix_MPT-0,5-5-2.54_1x05_P2.54mm_Horizontal")
     )
     (path "/964c1fd6-7dcf-4d74-b100-be5e91da66f6"
@@
     )
     (path "/aa1128dd-6f63-42e8-b1c8-5f38b2aacafb"
-      (reference "J104") (unit 1) (value "B1 C B2") (footprint "TerminalBlock_TE-Connectivity:TerminalBlock_TE_282834-3_1x03_P2.54mm_Horizontal")
+      (reference "J104") (unit 1) (value "B2 C B1") (footprint "TerminalBlock_TE-Connectivity:TerminalBlock_TE_282834-3_1x03_P2.54mm_Horizontal")
     )
     (path "/72f30a49-be47-4002-8fc7-9dc71c615793"
@@
     )
     (path "/3ad063d5-f655-45c2-8ae4-b0eef3b2ea53"
-      (reference "J107") (unit 1) (value "Servo 4") (footprint "Connector_PinHeader_2.54mm:PinHeader_1x03_P2.54mm_Vertical")
+      (reference "J107") (unit 1) (value "Sv 4") (footprint "Connector_PinHeader_2.54mm:PinHeader_1x03_P2.54mm_Vertical")
     )
     (path "/4fa36ec3-5569-4faf-a94f-4523bbaec2ab"
-      (reference "J108") (unit 1) (value "Servo 3") (footprint "Connector_PinHeader_2.54mm:PinHeader_1x03_P2.54mm_Vertical")
+      (reference "J108") (unit 1) (value "Sv 3") (footprint "Connector_PinHeader_2.54mm:PinHeader_1x03_P2.54mm_Vertical")
     )
     (path "/cfdc3bc5-ddc6-40cc-8cf4-e905dd0e45bb"
-      (reference "J109") (unit 1) (value "Servo 2") (footprint "Connector_PinHeader_2.54mm:PinHeader_1x03_P2.54mm_Vertical")
+      (reference "J109") (unit 1) (value "Sv 2") (footprint "Connector_PinHeader_2.54mm:PinHeader_1x03_P2.54mm_Vertical")
     )
     (path "/7cdb555d-8cef-4c84-b29f-bf59fa4cf452"
-      (reference "J110") (unit 1) (value "Servo 1") (footprint "Connector_PinHeader_2.54mm:PinHeader_1x03_P2.54mm_Vertical")
+      (reference "J110") (unit 1) (value "Sv 1") (footprint "Connector_PinHeader_2.54mm:PinHeader_1x03_P2.54mm_Vertical")
     )
     (path "/8861d1a1-8606-4193-916a-eb139c274d56"

Commit message: Add Activity LEDs.
Parts:
- added D103: ACT1, LED_SMD:LED_0603_1608Metric, symbol Device:LED
- added D104: ACT2, LED_SMD:LED_0603_1608Metric, symbol Device:LED
- added R109, R110: 130, Resistor_SMD:R_0603_1608Metric, symbol Device:R
Connections:
- net +3V3: now also R109.1, R110.1
- net A0: now also D104.2 (A)
- net A1: now also D103.2 (A)
- new net: D103.1 (K), R109.2
- new net: D104.1 (K), R110.2
- no-connect marks 16 -> 14
Changed lines of the file:
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@@
   (junction (at 31.75 46.99) (diameter 1.016) (color 0 0 0 0)
+  )
+  (junction (at 15.24 39.37) (diameter 0) (color 0 0 0 0)
   )
   (junction (at 225.425 137.795) (diameter 0) (color 0 0 0 0)
@@
   (no_connect (at 21.59 67.31))
   (no_connect (at 219.075 133.985))
-  (no_connect (at 21.59 62.23))
   (no_connect (at 219.075 131.445))
   (no_connect (at 273.685 119.38))
@@
   (no_connect (at 74.93 29.21))
   (no_connect (at 34.29 31.75))
-  (no_connect (at 21.59 59.69))
   (wire (pts (xy 260.35 20.32) (xy 263.525 20.32))
     (stroke (width 0) (type default) (color 0 0 0 0))
@@
     (stroke (width 0) (type default) (color 0 0 0 0))
   )
+  (wire (pts (xy 15.24 36.195) (xy 15.24 39.37))
+    (stroke (width 0) (type default) (color 0 0 0 0))
+  )
   (wire (pts (xy 62.23 44.45) (xy 74.93 44.45))
     (stroke (width 0) (type solid) (color 0 0 0 0))
@@
     (stroke (width 0) (type default) (color 0 0 0 0))
   )
+  (wire (pts (xy 15.24 55.88) (xy 15.24 62.23))
+    (stroke (width 0) (type default) (color 0 0 0 0))
+  )
   (wire (pts (xy 31.75 44.45) (xy 31.75 46.99))
     (stroke (width 0) (type solid) (color 0 0 0 0))
@@
     (stroke (width 0) (type default) (color 0 0 0 0))
   )
+  (wire (pts (xy 19.685 55.88) (xy 19.685 59.69))
+    (stroke (width 0) (type default) (color 0 0 0 0))
+  )
   (wire (pts (xy 242.57 154.94) (xy 242.57 111.76))
     (stroke (width 0) (type default) (color 0 0 0 0))
@@
     (stroke (width 0) (type default) (color 0 0 0 0))
   )
+  (wire (pts (xy 15.24 39.37) (xy 19.685 39.37))
+    (stroke (width 0) (type default) (color 0 0 0 0))
+  )
   (wire (pts (xy 31.75 26.67) (xy 31.75 39.37))
     (stroke (width 0) (type solid) (color 0 0 0 0))
@@
     (stroke (width 0) (type default) (color 0 0 0 0))
   )
-  (wire (pts (xy 34.29 59.69) (xy 21.59 59.69))
-    (stroke (width 0) (type solid) (color 0 0 0 0))
-  )
   (wire (pts (xy 62.23 39.37) (xy 74.93 39.37))
     (stroke (width 0) (type solid) (color 0 0 0 0))
@@
     (stroke (width 0) (type solid) (color 0 0 0 0))
   )
-  (wire (pts (xy 21.59 62.23) (xy 34.29 62.23))
-    (stroke (width 0) (type solid) (color 0 0 0 0))
-  )
   (wire (pts (xy 109.22 135.255) (xy 109.22 163.195))
     (stroke (width 0) (type default) (color 0 0 0 0))
@@
     (stroke (width 0) (type default) (color 0 0 0 0))
   )
+  (wire (pts (xy 15.24 62.23) (xy 34.29 62.23))
+    (stroke (width 0) (type default) (color 0 0 0 0))
+  )
   (wire (pts (xy 133.985 100.33) (xy 133.985 121.92))
     (stroke (width 0) (type default) (color 0 0 0 0))
@@
     (stroke (width 0) (type solid) (color 0 0 0 0))
   )
+  (wire (pts (xy 15.24 46.99) (xy 15.24 48.26))
+    (stroke (width 0) (type default) (color 0 0 0 0))
+  )
+  (wire (pts (xy 19.685 46.99) (xy 19.685 48.26))
+    (stroke (width 0) (type default) (color 0 0 0 0))
+  )
   (wire (pts (xy 215.9 30.48) (xy 215.9 34.29))
     (stroke (width 0) (type default) (color 0 0 0 0))
@@
   )
   (wire (pts (xy 247.015 154.94) (xy 247.015 158.75))
+    (stroke (width 0) (type default) (color 0 0 0 0))
+  )
+  (wire (pts (xy 19.685 59.69) (xy 34.29 59.69))
     (stroke (width 0) (type default) (color 0 0 0 0))
   )
@@
     (pin "14")
   )
+  (symbol (lib_id "Device:LED") (at 15.24 52.07 270) (unit 1)
+    (in_bom yes) (on_board yes)
+    (property "Reference" "D103" (id 0) (at 17.78 49.2124 90)
+      (effects (font (size 1.27 1.27)) (justify left))
+    )
+    (property "Value" "ACT1" (id 1) (at 13.335 55.245 90)
+      (effects (font (size 1.27 1.27)) (justify left))
+    )
+    (property "Footprint" "LED_SMD:LED_0603_1608Metric" (id 2) (at 15.24 52.07 0)
+      (effects (font (size 1.27 1.27)) hide)
+    )
+    (property "Datasheet" "~" (id 3) (at 15.24 52.07 0)
+      (effects (font (size 1.27 1.27)) hide)
+    )
+    (pin "1")
+    (pin "2")
+  )
+  (symbol (lib_id "Device:R") (at 19.685 43.18 0) (unit 1)
+    (in_bom yes) (on_board yes) (fields_autoplaced)
+    (property "Reference" "R110" (id 0) (at 21.59 41.9099 0)
+      (effects (font (size 1.27 1.27)) (justify left))
+    )
+    (property "Value" "130" (id 1) (at 21.59 44.4499 0)
+      (effects (font (size 1.27 1.27)) (justify left))
+    )
+    (property "Footprint" "Resistor_SMD:R_0603_1608Metric" (id 2) (at 17.907 43.18 90)
+      (effects (font (size 1.27 1.27)) hide)
+    )
+    (property "Datasheet" "~" (id 3) (at 19.685 43.18 0)
+      (effects (font (size 1.27 1.27)) hide)
+    )
+    (pin "1")
+    (pin "2")
+  )
   (symbol (lib_id "power:GND") (at 225.425 137.795 0) (unit 1)
     (in_bom yes) (on_board yes)
@@
     (property "Datasheet" "" (id 3) (at 268.605 26.035 0))
     (pin "1")
+  )
+  (symbol (lib_id "Device:R") (at 15.24 43.18 0) (unit 1)
+    (in_bom yes) (on_board yes) (fields_autoplaced)
+    (property "Reference" "R109" (id 0) (at 17.145 41.9099 0)
+      (effects (font (size 1.27 1.27)) (justify left))
+    )
+    (property "Value" "130" (id 1) (at 17.145 44.4499 0)
+      (effects (font (size 1.27 1.27)) (justify left))
+    )
+    (property "Footprint" "Resistor_SMD:R_0603_1608Metric" (id 2) (at 13.462 43.18 90)
+      (effects (font (size 1.27 1.27)) hide)
+    )
+    (property "Datasheet" "~" (id 3) (at 15.24 43.18 0)
+      (effects (font (size 1.27 1.27)) hide)
+    )
+    (pin "1")
+    (pin "2")
   )
   (symbol (lib_id "STM32F303-RIR4-rescue:+12V") (at 123.19 29.845 0) (unit 1)
@@
     (pin "9")
   )
+  (symbol (lib_id "Device:LED") (at 19.685 52.07 270) (unit 1)
+    (in_bom yes) (on_board yes)
+    (property "Reference" "D104" (id 0) (at 22.86 49.2124 90)
+      (effects (font (size 1.27 1.27)) (justify left))
+    )
+    (property "Value" "ACT2" (id 1) (at 18.415 55.245 90)
+      (effects (font (size 1.27 1.27)) (justify left))
+    )
+    (property "Footprint" "LED_SMD:LED_0603_1608Metric" (id 2) (at 19.685 52.07 0)
+      (effects (font (size 1.27 1.27)) hide)
+    )
+    (property "Datasheet" "~" (id 3) (at 19.685 52.07 0)
+      (effects (font (size 1.27 1.27)) hide)
+    )
+    (pin "1")
+    (pin "2")
+  )
   (symbol (lib_id "STM32F303-RIR4-rescue:+12V") (at 128.905 93.98 0) (unit 1)
     (in_bom yes) (on_board yes)
@@
     (pin "9")
   )
+  (symbol (lib_id "power:+3V3") (at 15.24 36.195 0) (unit 1)
+    (in_bom yes) (on_board yes)
+    (property "Reference" "#PWR0120" (id 0) (at 15.24 40.005 0)
+      (effects (font (size 1.27 1.27)) hide)
+    )
+    (property "Value" "+3.3V" (id 1) (at 15.621 33.147 90)
+      (effects (font (size 1.27 1.27)) (justify left))
+    )
+    (property "Footprint" "" (id 2) (at 15.24 36.195 0))
+    (property "Datasheet" "" (id 3) (at 15.24 36.195 0))
+    (pin "1")
+  )
   (symbol (lib_id "STM32F303-RIR4-rescue:ASSR-1218") (at 208.28 27.94 0) (unit 1)
     (in_bom yes) (on_board yes)
@@
       (reference "#PWR0119") (unit 1) (value "+5V") (footprint "")
     )
+    (path "/74405455-216b-4710-a117-4b345b87165d"
+      (reference "#PWR0120") (unit 1) (value "+3.3V") (footprint "")
+    )
     (path "/ad075a32-e96f-4652-bef0-90f728f36fff"
       (reference "C101") (unit 1) (value ".1 uf") (footprint "Capacitor_SMD:C_0603_1608Metric")
@@
       (reference "D102") (unit 1) (value "TX") (footprint "LED_SMD:LED_0603_1608Metric")
     )
+    (path "/11ee97cc-ce53-4b96-a677-5039ac9f2dd5"
+      (reference "D103") (unit 1) (value "ACT1") (footprint "LED_SMD:LED_0603_1608Metric")
+    )
+    (path "/69f30c7e-597f-4c15-b830-2b1b0fcf8cd8"
+      (reference "D104") (unit 1) (value "ACT2") (footprint "LED_SMD:LED_0603_1608Metric")
+    )
     (path "/00000000-0000-0000-0000-000056d71773"
       (reference "J1") (unit 1) (value "Power") (footprint "Connector_PinSocket_2.54mm:PinSocket_1x08_P2.54mm_Vertical")
@@
       (reference "R108") (unit 1) (value "5K to 20K") (footprint "Resistor_THT:R_Axial_DIN0204_L3.6mm_D1.6mm_P7.62mm_Horizontal")
     )
+    (path "/26267479-963d-4e50-bf5c-e68c32c61d39"
+      (reference "R109") (unit 1) (value "130") (footprint "Resistor_SMD:R_0603_1608Metric")
+    )
+    (path "/1406d2d2-5f3e-472b-bdec-f6e54481bb02"
+      (reference "R110") (unit 1) (value "130") (footprint "Resistor_SMD:R_0603_1608Metric")
+    )
     (path "/bdb711b3-72f8-4503-8ae0-33630d570bf9"

Commit message: Update part numbers, etc.
Parts:
- C101: Manufacturer (none) -> KEMET; Manufacturer Part Number (none) -> C0603C104M5RACTU; Mouser Part Number 710-885012206095 -> 80-C0603C104M5R
- C102: Manufacturer (none) -> Nichicon; Manufacturer Part Number (none) -> UUD1C150MCL1GS; Mouser Part Number 710-865080340002 -> 647-UUD1C150MCL
- D101: LCSC C7083723 -> (none); MPN Lumex SML-LX0603YW-TR -> (none); Manufacturer (none) -> Lumex; Manufacturer Part Number (none) -> SML-LX0603YW-TR
- D102: LCSC C5354817 -> (none); MPN Lumex SML-LX0603IW-TR -> (none); Manufacturer (none) -> Lumex; Manufacturer Part Number (none) -> SML-LX0603IW-TR
- D103: Manufacturer (none) -> Lumex; Manufacturer Part Number (none) -> SML-LX0603IW-TR; Mouser Part Number (none) -> 710-150060SS75000
- D104: Manufacturer (none) -> Lumex; Manufacturer Part Number (none) -> SML-LX0603YW-TR; Mouser Part Number (none) -> 710-150060YS75000
- R101, R102: LCSC C859411 -> (none); MPN YAGEO RE0603FRE07330RL -> (none); Manufacturer (none) -> YAGEO; Manufacturer Part Number (none) -> RE0603FRE07330RL
- R103, R104: value 390 -> 130; LCSC C228185 -> (none); MPN YAGEO AC0603JR-07390RL -> (none); Manufacturer (none) -> YAGEO; Manufacturer Part Number (none) -> AC0603JR-07130RL; Mouser Part Number 603-AC0603JR-07390RL -> 603-AC0603JR-07130RL
- R109: Manfacturer Part Number (none) -> AC0603JR-07130RL; Manufacturer (none) -> YAGEO; Mouser Part Number (none) -> 603-AC0603JR-07130RL
- R110: Manufacturer (none) -> YAGEO; Manufacturer Part Number (none) -> AC0603JR-07130RL; Mouser Part Number (none) -> 603-AC0603JR-07130RL
- U101: LCSC C141521 -> (none); MPN TOSHIBA TBD62064AFG,EL -> (none); Manufacturer (none) -> TOSHIBA; Manufacturer Part Number (none) -> TBD62064AFG,EL
- U102, U103: LCSC C624948 -> (none); MPN Microchip TC4428ACOA713 -> (none); Manufacturer (none) -> Microchip; Manufacturer Part Number (none) -> TC4428ACOA713
- U104, U105: LCSC C19844354 -> (none); MPN OMRON G3VM-61VY4(TR05) -> (none); Manufacturer (none) -> OMRON; Manufacturer Part Number (none) -> G3VM-61VY4(TR05)
- U106: LCSC C5145450 -> (none); MPN HANSCHIP semiconductor LM358DRG -> (none); Manufacturer (none) -> HANSCHIP semiconductor; Manufacturer Part Number (none) -> LM358DRG
- U107: Manufacturer (none) -> Texas Instruments; Manufacturer Part Number (none) -> TCAN332DR

Commit message: Complete PCBWay BOM.
Parts:
- C101: MPN (none) -> KEMET C0603C104M5RACTU
- C102: MPN (none) -> Nichicon UUD1C150MCL1GS
- D101, D104: MPN (none) -> Lumex SML-LX0603YW-TR
- D102, D103: MPN (none) -> Lumex SML-LX0603IW-TR
- J1, J2, J3, J4: now left out of the parts list
- R101, R102: MPN (none) -> YAGEO RE0603FRE07330RL
- R103, R104, R110: MPN (none) -> YAGEO AC0603JR-07130RL
- R109: MPN (none) -> YAGEO AC0603JR-07130RL; Manfacturer Part Number AC0603JR-07130RL -> (none); Manufacturer Part Number (none) -> AC0603JR-07130RL
- U101: MPN (none) -> TOSHIBA TBD62064AFG,EL
- U102, U103: MPN (none) -> Microchip TC4428ACOA713
- U104, U105: MPN (none) -> OMRON G3VM-61VY4(TR05)
- U106: MPN (none) -> HANSCHIP semiconductor LM358DRG
- U107: MPN (none) -> Texas Instruments TCAN332DR
